File: circuit/RedMyst.kicad_pcb (KiCad board)
At the start: 2 copper layers, 51 parts, among them J1 CONN_01X09, J2 CONN_01X03, SW1 IN/OUT, SW2 WP, U1 LM1117, U2 FV-1, U3 24LC32A, U4 SW_1P8T, Y1 32768Hz

Commit message: RedMyst continued
Parts:
- removed C1, C2: 3.3µf, myAmp:CPOL_D4_P1.5
- removed C10, C7: 1nF, myAmp:C_1206
- removed C11, C13: 100nF, myAmp:C_1206
- removed C12, C3, C6, C9: 1µF, myAmp:C_1206
- removed C14: 15pF, myAmp:C_0805
- removed C4, C5: 2.2nF, myAmp:C_1206
- removed C8: 100µf, myAmp:CPOL_D8_P3.5
- removed D1: CLIP, myAmp:LED_D3.0mm
- removed D10, D2, D3, D4, D5, D6, D7, D8, D9: BAT43, myAmp:DO35
- removed D11: PWR, myAmp:LED_D3.0mm
- removed J1: CONN_01X09, myAmp:PIN_1x09
- removed J2: CONN_01X03, myAmp:PIN_1x03
- removed R1, R2, R3, R4: 1K, myAmp:R_10MM
- removed R10, R11, R13: 100K, myAmp:R_10MM
- removed R12, R9: 20K, myAmp:R_10MM
- removed R14: 100, myAmp:R_10MM
- removed R5, R6: 10K, myAmp:R_10MM
- removed R7, R8: 100, myAmp:R_0805
- removed RV1, RV2, RV3: 50K, myAmp:ALPS_RK09K113
- removed SW1: IN/OUT, myAmp:JUMPER
- removed SW2: WP, myAmp:JUMPER
- removed U1: LM1117, myAmp:SOT-223
- removed U2: FV-1, myAmp:SOIC-28_7.5x17.9mm_Pitch1.27mm
- removed U3: 24LC32A, myAmp:DIP-8
- removed U4: SW_1P8T, myAmp:SR17B1815F89N
- removed Y1: 32768Hz, myAmp:QUARTZ_85SMX
Routing:
- net +3V3: track 54.3 -> 0.00 mm
- net Net-(D2-Pad1): track 52.7 -> 0.00 mm
- net Net-(D6-Pad1): track 51.9 -> 0.00 mm
- net Net-(D10-Pad1): track 44.7 -> 0.00 mm
- net Net-(RV2-Pad2): track 42.0 -> 0.00 mm
- net MID: track 36.8 -> 0.00 mm
- net Net-(RV3-Pad2): track 32.0 -> 0.00 mm
- net Net-(RV1-Pad2): track 31.8 -> 0.00 mm
- net SDA: track 31.5 -> 0.00 mm
- net SCL: track 23.5 -> 0.00 mm
- net Net-(R9-Pad1): track 20.6 -> 0.00 mm
- net RIN: track 20.1 -> 0.00 mm
- net LIN: track 16.1 -> 0.00 mm
- net Net-(D10-Pad2): track 12.9 -> 0.00 mm
- net Net-(C1-Pad2): track 12.5 -> 0.00 mm
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Other:
- board text removed: "3V3"
- board text removed: "GND"
- board text removed: "LIN"
- board text removed: "MID"
- board text removed: "RIN"
- board text removed: "SCL"
- board text removed: "SDA"
- board text removed: "VCC"
- board text removed: "WP"

Commit message: RedMyst continued...
Parts:
- added BT1: Battery, myAmp:BATTERY, F.Cu at (113.0, 16.0)
- added C1: 1µF, myAmp:C_1206, F.Cu at (83.1, 49.3)
- added C10: 100nF, myAmp:C_5MM, F.Cu at (62.3, 63.8)
- added C11: 100nF, myAmp:C_1206, F.Cu at (75.4, 55.1)
- added C12: 1µF, myAmp:C_1206, F.Cu at (101.5, 27.7)
- added C13: 1nF, myAmp:C_0805, F.Cu at (104.1, 18.5)
- added C14: 100nF, myAmp:C_1206, F.Cu at (77.3, 52.2)
- added C15: 47nF, myAmp:C_5MM, F.Cu at (68.9, 56.3)
- added C16: 220μF, myAmp:CPOL_D6.3_P2.5, F.Cu at (61.6, 58.4)
- added C17: 15pF, myAmp:C_0805, F.Cu at (76.4, 67.6)
- added C18: 1µF, myAmp:C_1206, F.Cu at (75.4, 58.0)
- added C19: 100µf, myAmp:CPOL_D8_P3.5, F.Cu at (86.5, 25.4)
- added C2: 10nF, myAmp:C_1206, F.Cu at (93.9, 38.6)
- added C20: 1µF, myAmp:C_1206, F.Cu at (61.7, 66.8)
- added C21: 100nF, myAmp:C_0805, F.Cu at (50.8, 90.2)
- added C22: 100nF, myAmp:C_0805, F.Cu at (78.7, 46.2)
- added C23: 1µF, myAmp:C_1206, F.Cu at (101.5, 24.8)
- added C24: 1µF, myAmp:C_1206, F.Cu at (86.8, 41.8)
- added C25: 100nF, myAmp:C_1206, F.Cu at (107.3, 27.7)
- added C26: 22pF, myAmp:C_2.5MM, F.Cu at (44.8, 72.3)
- added C27: 100μF, myAmp:CPOL_D6.3_P2.5, F.Cu at (55.0, 65.9)
- added C28: 100nF, myAmp:C_1206, F.Cu at (77.3, 49.3)
- added C29: 1nF, myAmp:C_1206, F.Cu at (95.2, 32.1)
- added C3: 10nF, myAmp:C_1206, F.Cu at (110.6, 19.3)
- added C30: 100μF, myAmp:CPOL_D6.3_P2.5, F.Cu at (114.4, 10.4)
- added C31: 100nF, myAmp:C_1206, F.Cu at (85.1, 46.0)
- added C32: 1nF, myAmp:C_1206, F.Cu at (95.2, 35.0)
- added C33: 680nF, myAmp:C_FILM_5MM, F.Cu at (81.0, 33.5)
- added C34: 22pF, myAmp:C_2.5MM, F.Cu at (53.4, 60.7)
- added C35: 680nF, myAmp:C_FILM_5MM, F.Cu at (106.5, 8.99)
- added C36: 1μF, myAmp:C_1206, F.Cu at (79.8, 37.3)
- added C37: 1μF, myAmp:C_1206, F.Cu at (67.5, 68.1)
- added C38: 680nF, myAmp:C_FILM_5MM, F.Cu at (46.7, 68.8)
- added C39: 220nF, myAmp:C_1206, F.Cu at (74.6, 61.0)
- added C4: 1μF, myAmp:C_FILM_5MM, F.Cu at (32.4, 88.3)
- added C40: 220nF, myAmp:C_1206, F.Cu at (91.0, 44.7)
- added C41: 1μF, myAmp:C_1206, F.Cu at (92.7, 41.8)
- added C42: 220nF, myAmp:C_1206, F.Cu at (101.5, 30.6)
- added C43: 680nF, myAmp:C_FILM_5MM, F.Cu at (71.0, 45.0)
- added C44: 1μF, myAmp:C_1206, F.Cu at (68.8, 65.2)
- added C45: 220nF, myAmp:C_1206, F.Cu at (68.8, 62.2)
- added C46: 1μF, myAmp:C_1206, F.Cu at (61.7, 69.8)
- added C47: 1μF, myAmp:C_1206, F.Cu at (107.3, 24.8)
- added C48: 100nF, myAmp:C_5MM, F.Cu at (87.5, 38.7)
- added C5: 1nF, myAmp:C_1206, F.Cu at (116.4, 19.3)
- added C6: 250pF, myAmp:C_5MM, F.Cu at (104.1, 21.7)
- added C7: 220μF, myAmp:CPOL_D6.3_P2.5, F.Cu at (94.8, 26.9)
- added C8: 1µF, myAmp:C_1206, F.Cu at (68.3, 59.3)
- added C9: 1nF, myAmp:C_0805, F.Cu at (47.0, 95.9)
- added D1: 1N4148, myAmp:DO35, F.Cu at (50.4, 49.5)
- added D2: 1N4773a, myAmp:DO41, F.Cu at (14.0, 97.2)
- added D3: 1N4773a, myAmp:DO41, F.Cu at (14.0, 94.0)
- added D4: CLIP, myAmp:LED_D3.0mm, F.Cu at (112.8, 23.4)
- added D5: 1N4148, myAmp:DO35, F.Cu at (84.5, 19.6)
- added D6: PWR, myAmp:LED_D3.0mm, F.Cu at (106.9, 31.8)
- added D7: FAULT, myAmp:LED_D3.0mm, F.Cu at (100.7, 34.7)
- added D8: PWR, myAmp:LED_D3.0mm, F.Cu at (82.8, 53.3)
- added J1: JACK_MONO, myAmp:JACK_CL13106, F.Cu at (12.1, 81.9)
- added J2: CONN_01X03, myAmp:PIN_1x03, F.Cu at (71.9, 40.9)
- added J3: HOLE, myAmp:MountingHole, F.Cu at (96.0, 96.0)
- added J4: HOLE, myAmp:MountingHole, F.Cu at (96.0, 4.00)
- added J5: HOLE, myAmp:MountingHole, F.Cu at (4.00, 4.00)
- added J6: HOLE, myAmp:MountingHole, F.Cu at (4.00, 96.0)
- added L1: 10μH, myAmp:COILCRAFT_DR0810, F.Cu at (86.3, 12.5)
- added L2: 10μH, myAmp:COILCRAFT_DR0810, F.Cu at (34.3, 57.6)
- added L3: 10μH, myAmp:COILCRAFT_DR0810, F.Cu at (51.1, 42.4)
- added L4: 10μH, myAmp:COILCRAFT_DR0810, F.Cu at (73.6, 16.2)
- added Q1: MMBFJ201, myAmp:SOT-23, F.Cu at (26.7, 89.5)
- added Q2: BC547, myAmp:TO-92_Inline_Wide, F.Cu at (70.6, 50.5)
- added Q3: BC557, myAmp:TO-92_Inline_Wide, F.Cu at (106.1, 14.5)
- added R1: 1K, myAmp:R_1206, F.Cu at (109.2, 35.6)
- added R10: 1M, myAmp:R_1206, F.Cu at (23.5, 96.5)
- added R11: 1, myAmp:R_1206, F.Cu at (28.6, 96.5)
- added R12: 1K, myAmp:R_1206, F.Cu at (39.4, 95.9)
- added R13: 10K, myAmp:R_1206, F.Cu at (41.9, 95.9)
- added R14: 10, myAmp:R_1206, F.Cu at (100.8, 45.8)
- added R15: 100, myAmp:R_1206, F.Cu at (106.8, 38.0)
- added R16: 10K, myAmp:R_1206, F.Cu at (102.8, 38.5)
- added R17: 1K, myAmp:R_1206, F.Cu at (118.1, 15.4)
- added R18: 4K7, myAmp:R_1206, F.Cu at (92.8, 49.8)
- added R19: 10K, myAmp:R_1206, F.Cu at (96.8, 45.5)
- added R2: 1K, myAmp:R_1206, F.Cu at (96.8, 47.9)
- added R20: 10K, myAmp:R_1206, F.Cu at (85.0, 57.2)
- added R21: 10K, myAmp:R_1206, F.Cu at (71.4, 70.8)
- added R22: 10K, myAmp:R_1206, F.Cu at (78.4, 63.6)
- added R23: 10K, myAmp:R_1206, F.Cu at (87.4, 52.6)
- added R24: 10K, myAmp:R_1206, F.Cu at (92.8, 47.4)
- added R25: 10K, myAmp:R_1206, F.Cu at (79.5, 61.1)
- added R26: 100, myAmp:R_1206, F.Cu at (101.7, 41.0)
- added R27: 10K, myAmp:R_1206, F.Cu at (117.3, 24.4)
- added R28: 10K, myAmp:R_1206, F.Cu at (112.2, 29.6)
- added R29: 10K, myAmp:R_1206, F.Cu at (105.2, 35.6)
- added R3: 1, myAmp:R_1206, F.Cu at (26.0, 96.5)
- added R30: 10K, myAmp:R_1206, F.Cu at (72.4, 67.8)
- added R31: 10K, myAmp:R_1206, F.Cu at (112.2, 27.2)
- added R32: 10K, myAmp:R_1206, F.Cu at (117.3, 22.0)
- added R33: 10K, myAmp:R_1206, F.Cu at (109.6, 61.6)
- added R34: 10K, myAmp:R_1206, F.Cu at (60.0, 72.4)
- added R35: 2K2, myAmp:R_1206, F.Cu at (91.4, 52.6)
- added R36: 2K2, myAmp:R_1206, F.Cu at (111.5, 32.0)
- added R4: 1K, myAmp:R_1206, F.Cu at (116.2, 29.6)
- added R5: 4K7, myAmp:R_1206, F.Cu at (101.7, 43.4)
- added R6: 100, myAmp:R_1206, F.Cu at (116.2, 27.2)
- added R7: 100K, myAmp:R_1206, F.Cu at (82.4, 63.5)
- added R8: 1M, myAmp:R_1206, F.Cu at (36.8, 95.9)
- added R9: 10, myAmp:R_1206, F.Cu at (89.0, 55.0)
- added RN1: 100, myAmp:R_Array_x4_1206, F.Cu at (80.6, 57.9)
- added RN2: 100, myAmp:R_Array_x4_1206, F.Cu at (67.0, 71.5)
- added RN3: 100, myAmp:R_Array_x4_1206, F.Cu at (74.1, 64.4)
- added RN4: 100, myAmp:R_Array_x4_1206, F.Cu at (88.4, 49.5)
- added RV1: 250K, myAmp:ALPS_RK09K113, F.Cu at (31.3, 31.6)
- added RV2: 50K, myAmp:ALPS_RK09K113, F.Cu at (38.3, 50.4)
- added RV3: 50K, myAmp:ALPS_RK09K113, F.Cu at (60.8, 19.7)
- added RV4: 50K, myAmp:ALPS_RK09K113, F.Cu at (21.5, 62.0)
- added RV5: 250K, myAmp:ALPS_RK09K113, F.Cu at (49.5, 30.9)
- added RV6: 10K, myAmp:ALPS_RK09K113, F.Cu at (22.3, 43.3)
- added S1: LEFT, myAmp:SPKR_5MM, F.Cu at (76.3, 26.6)
- added S2: RIGHT, myAmp:SPKR_5MM, F.Cu at (20.2, 68.0)
- added SS1: SEVSEG, myAmp:7seg_14.2mm, F.Cu at (93.3, 73.7)
- added SS2: SEVSEG, myAmp:7seg_14.2mm, F.Cu at (106.7, 73.7)
- added SW1: ROT_SW, myAmp:ROT_ENC, F.Cu at (30.9, 16.2)
- added SW2: ON/OFF, myAmp:SW_TINY, F.Cu at (46.9, 64.6)
- added T1: DSP_IN, myAmp:TestPad, F.Cu at (29.9, 50.3)
- added U1: NE5532, myAmp:SOIC-8_3.9x4.9mm_P1.27mm, F.Cu at (41.3, 88.3)
- added U10: 74164, myAmp:SOIC-14_3.9x8.7mm_P1.27mm, F.Cu at (84.5, 87.6)
- added U11: TPA3136D2, myAmp:HTSSOP-28_4.4x9.7mm_Pitch0.65mm_ThermalPad, F.Cu at (63.0, 36.6)
- added U2: NE5532, myAmp:SOIC-8_3.9x4.9mm_P1.27mm, F.Cu at (62.1, 51.5)
- added U3: TLE2426, myAmp:TO-92_Inline_Wide, F.Cu at (80.1, 42.2)
- added U4: FV-1, myAmp:SOIC-28_7.5x17.9mm_Pitch1.27mm, F.Cu at (7.05, 44.9)
- added U5: LM1117, myAmp:SOT-223, F.Cu at (72.2, 35.1)
- added U6: 24LC32A, myAmp:DIP-8, F.Cu at (97.2, 11.7)
- added U7: 74164, myAmp:SOIC-14_3.9x8.7mm_P1.27mm, F.Cu at (73.7, 85.7)
- added U8: AVR-ISP6, myAmp:AVR_ISP6, F.Cu at (57.7, 57.9)
- added U9: ATMEGA8-16AU, myAmp:TQFP-32_7x7mm_Pitch0.8mm, F.Cu at (45.6, 57.3)
- added Y1: 32768Hz, myAmp:QUARTZ_85SMX, F.Cu at (61.9, 45.2)
- added Y2: 8MHz, myAmp:Crystal_HC49-U_Vertical, F.Cu at (64.6, 28.0)
Other:
- board outline added: 100 x 100 mm
- copper layers 2 -> 4

Commit message: added alps 3d models
Parts:
- removed T1: DSP_IN, myAmp:TestPad
- added NB1: qo, myAmp:NET_BRK, F.Cu at (32.4, 96.5)
- added NB10: rs2o, myAmp:NET_BRK, F.Cu at (189.9, 63.5)
- added NB11: lmti, myAmp:NET_BRK, F.Cu at (-59.1, 53.3)
- added NB12: rmdi, myAmp:NET_BRK, F.Cu at (-59.1, 62.2)
- added NB13: rmao, myAmp:NET_BRK, F.Cu at (-78.7, 49.5)
- added NB14: rmai, myAmp:NET_BRK, F.Cu at (-78.7, 52.1)
- added NB15: rmti, myAmp:NET_BRK, F.Cu at (-59.1, 68.6)
- added NB16: lpi, myAmp:NET_BRK, F.Cu at (54.6, 24.1)
- added NB17: lni, myAmp:NET_BRK, F.Cu at (54.6, 26.7)
- added NB18: rni, myAmp:NET_BRK, F.Cu at (54.6, 34.3)
- added NB19: rpi, myAmp:NET_BRK, F.Cu at (54.6, 36.8)
- added NB2: a1o, myAmp:NET_BRK, F.Cu at (44.5, 96.5)
- added NB3: jo, myAmp:NET_BRK, F.Cu at (21.6, 96.5)
- added NB4: tso, myAmp:NET_BRK, F.Cu at (38.7, 81.3)
- added NB5: a2o, myAmp:NET_BRK, F.Cu at (33.0, 75.6)
- added NB6: rso, myAmp:NET_BRK, F.Cu at (193.0, 63.5)
- added NB7: lmdi, myAmp:NET_BRK, F.Cu at (-59.1, 47.0)
- added NB8: lmao, myAmp:NET_BRK, F.Cu at (-92.7, 50.2)
- added NB9: lmai, myAmp:NET_BRK, F.Cu at (34.9, 46.0)
- added RV7: 10K, myAmp:ALPS_RK09L_DBL, F.Cu at (-39.4, 57.8)
- added RV8: 10K, myAmp:ALPS_RK09L_DBL, F.Cu at (-25.4, 57.8)
- C10, C15, C48, C6: footprint myAmp:C_5MM -> myAmp:C_5MM_1206
- C13, C17, C21, C22, C9: footprint myAmp:C_0805 -> myAmp:C_1206
- C4: footprint myAmp:C_FILM_5MM -> myAmp:C_5MM_1206
- RV1, RV2, RV3, RV4, RV5, RV6: footprint myAmp:ALPS_RK09K113 -> myAmp:ALPS_RK09L
- U9: value ATMEGA8-16AU -> ATMEGA8
- moved RV4 188.2 mm to (207.0, 29.8)
- moved R32 174.5 mm to (-50.8, 68.6), turned to 90 degrees
- moved R27 173.1 mm to (-53.3, 53.3), turned to 270 degrees
- moved R31 170.6 mm to (-53.3, 68.6), turned to 270 degrees
- moved R28 164.7 mm to (-50.8, 53.3), turned to 90 degrees
- moved C22 164.4 mm to (-85.7, 45.7)
- moved C23 161.7 mm to (-55.9, 62.2), turned to 270 degrees
- moved R29 160.8 mm to (-53.3, 62.2), turned to 90 degrees
- moved U2 148.6 mm to (-86.5, 50.9)
- moved R24 146.1 mm to (-53.3, 47.0), turned to 90 degrees
- moved C24 145.2 mm to (-55.9, 68.6), turned to 90 degrees
- moved RV2 142.2 mm to (179.1, 29.8)
- moved U4 141.9 mm to (144.8, 10.8)
- moved RV3 132.6 mm to (193.0, 29.8)
- moved C18 131.7 mm to (-55.9, 47.0), turned to 270 degrees
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Connections:
- net Net-(C12-Pad2) renamed /MID
- C13 pad 1: /TONE_OUT -> Net-(C13-Pad1)
- C16 pad 1: VGND -> Net-(C16-Pad1)
- C18 pad 1: /FV_LOUT -> Net-(C18-Pad1)
- C20 pad 1: /TONE_OUT -> Net-(C20-Pad1)
- C23 pad 1: /FV_ROUT -> Net-(C23-Pad1)
- C24 pad 1: /TONE_OUT -> Net-(C24-Pad1)
- C41 pad 2: LOUT -> Net-(C41-Pad2)
- C44 pad 2: GND -> Net-(C44-Pad2)
- C46 pad 2: ROUT -> Net-(C46-Pad2)
- C47 pad 2: GND -> Net-(C47-Pad2)
- C48 pad 2: VGND -> Net-(C48-Pad2)
- C7 pad 2: VGND -> Net-(C16-Pad1)
- C9 pad 1: Net-(C6-Pad2) -> Net-(C9-Pad1)
- D1 pad 1: VGND -> Net-(C16-Pad1)
- D5 pad 2: VGND -> Net-(C16-Pad1)
- J1 pad 6: Net-(D2-Pad2) -> Net-(J1-Pad6)
- Q1 pad 1: Net-(C4-Pad2) -> Net-(NB1-Pad2)
- R13 pad 2: Net-(C6-Pad2) -> Net-(C9-Pad1)
- R14 pad 2: VGND -> Net-(C16-Pad1)
- R16 pad 2: /TONE_OUT -> Net-(C13-Pad1)
- R25 pad 2: Net-(R25-Pad2) -> Net-(NB9-Pad2)
- R28 pad 2: Net-(R25-Pad2) -> Net-(NB9-Pad2)
- R3 pad 1: Net-(C4-Pad2) -> Net-(NB1-Pad2)
- R30 pad 2: Net-(R30-Pad2) -> Net-(NB14-Pad2)
- R32 pad 2: Net-(R30-Pad2) -> Net-(NB14-Pad2)
- R9 pad 1: VGND -> Net-(C16-Pad1)
- RV1 pad 2: Net-(RV1-Pad2) -> Net-(NB4-Pad2)
- SS1 pad 10: Net-(RN2-Pad5) -> Net-(RN2-Pad8)
- SS1 pad 6: Net-(RN2-Pad8) -> Net-(RN2-Pad5)
- SS1 pad 7: Net-(RN2-Pad7) -> Net-(RN2-Pad6)
- SS1 pad 9: Net-(RN2-Pad6) -> Net-(RN2-Pad7)
- SS2 pad 10: Net-(RN4-Pad5) -> Net-(RN4-Pad8)
- SS2 pad 6: Net-(RN4-Pad8) -> Net-(RN4-Pad5)
- SS2 pad 7: Net-(RN4-Pad7) -> Net-(RN4-Pad6)
- SS2 pad 9: Net-(RN4-Pad6) -> Net-(RN4-Pad7)
- U1 pad 1: Net-(C6-Pad2) -> Net-(C9-Pad1)
- U1 pad 5: Net-(RV1-Pad2) -> Net-(NB4-Pad1)
- U1 pad 7: /TONE_OUT -> Net-(C13-Pad1)
- U10 pad 1: Net-(RN2-Pad4) -> Net-(RN2-Pad1)
- U10 pad 10: Net-(RN4-Pad1) -> Net-(RN4-Pad4)
- U10 pad 11: Net-(RN4-Pad2) -> Net-(RN4-Pad3)
- U10 pad 12: Net-(RN4-Pad3) -> Net-(RN4-Pad2)
- U10 pad 13: Net-(RN4-Pad4) -> Net-(RN4-Pad1)
- U10 pad 2: Net-(RN2-Pad4) -> Net-(RN2-Pad1)
- U2 pad 1: LOUT -> Net-(NB8-Pad2)
- U2 pad 2: Net-(R25-Pad2) -> Net-(NB9-Pad1)
- U2 pad 6: Net-(R30-Pad2) -> Net-(NB14-Pad1)
- U2 pad 7: ROUT -> Net-(NB13-Pad2)
- U3 pad 1: VGND -> Net-(C48-Pad2)
- U5 pad 3: (no net) -> VDD
- U7 pad 10: Net-(RN2-Pad1) -> Net-(RN2-Pad4)
- U7 pad 11: Net-(RN2-Pad2) -> Net-(RN2-Pad3)
- U7 pad 12: Net-(RN2-Pad3) -> Net-(RN2-Pad2)
- U7 pad 13: Net-(RN2-Pad4) -> Net-(RN2-Pad1)

Commit message: labels
Parts:
- moved RV4 41.9 mm to (165.1, 29.8)
- moved RV2 14.0 mm to (193.0, 29.8)
- moved RV3 14.0 mm to (179.1, 29.8)
Other:
- board text added: "bass"
- board text added: "master"
- board text added: "mid"
- board text added: "param 1"
- board text added: "param 2"
- board text added: "param 3"
- board text added: "treble"
- board text added: "wet/dry"

Commit message: localiced 3d models
Parts:
- moved C2 159.2 mm to (4.45, 47.6), turned to 270 degrees
- moved R1 156.0 mm to (6.99, 47.6), turned to 270 degrees
- moved R2 152.8 mm to (9.53, 47.6), turned to 90 degrees
- moved C3 149.6 mm to (12.1, 47.6), turned to 90 degrees
- moved C8 146.5 mm to (14.6, 47.6), turned to 90 degrees
- moved C11 143.3 mm to (17.1, 47.6), turned to 90 degrees
- moved C12 140.3 mm to (4.01, 61.0)
- moved C1 139.3 mm to (9.73, 67.9)
- moved R4 139.3 mm to (9.78, 65.4)
- moved R19 136.9 mm to (21.6, 48.9), turned to 90 degrees
- moved D4 135.8 mm to (3.17, 67.3), turned to 270 degrees
- moved R20 133.8 mm to (24.1, 48.9), turned to 270 degrees
- moved U4 133.6 mm to (19.7, 57.8), turned to 90 degrees
- moved R15 132.1 mm to (14.6, 66.7), turned to 90 degrees
- moved R22 130.8 mm to (26.7, 48.9), turned to 90 degrees
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Connections:
- C14 pad 1: Net-(C14-Pad1) -> GND
- J3 pad 1: (no net) -> Net-(J3-Pad1)
- J4 pad 1: (no net) -> Net-(J4-Pad1)
- J5 pad 1: (no net) -> Net-(J5-Pad1)
- J6 pad 1: (no net) -> Net-(J6-Pad1)
- U11 pad 13: (no net) -> Net-(U11-Pad13)
- U11 pad 5: (no net) -> Net-(U11-Pad5)
- U11 pad 6: (no net) -> Net-(U11-Pad6)
- U4 pad 6: Net-(C14-Pad1) -> +3V3
- U4 pad 8: Net-(C14-Pad1) -> +3V3
- U9 pad 1: (no net) -> Net-(U9-Pad1)
- U9 pad 19: (no net) -> Net-(U9-Pad19)
- U9 pad 2: (no net) -> Net-(U9-Pad2)
- U9 pad 22: (no net) -> Net-(U9-Pad22)
- U9 pad 32: (no net) -> Net-(U9-Pad32)

Commit message: layout done; starting routing
Parts:
- removed BT1: Battery, myAmp:BATTERY
- removed D6: PWR, myAmp:LED_D3.0mm
- removed NB11: lmti, myAmp:NET_BRK
- removed NB12: rmdi, myAmp:NET_BRK
- removed NB13: rmao, myAmp:NET_BRK
- removed NB14: rmai, myAmp:NET_BRK
- removed NB15: rmti, myAmp:NET_BRK
- removed NB7: lmdi, myAmp:NET_BRK
- removed NB8: lmao, myAmp:NET_BRK
- removed NB9: lmai, myAmp:NET_BRK
- removed R26: 100, myAmp:R_1206
- added J7: Barrel_Jack_Switch, myAmp:POWER_JACK_2.1mm, F.Cu at (93.3, 79.4)
- C19: value 100µf -> 10µf; footprint myAmp:CPOL_D8_P3.5 -> myAmp:CPOL_D4_P1.5
- C26, C34: footprint myAmp:C_2.5MM -> myAmp:C_1206
- C27, C30: footprint myAmp:CPOL_D6.3_P2.5 -> myAmp:CPOL_D8_P3.5
- SW2: footprint myAmp:SW_TINY -> myAmp:ESP2010_switch
- moved NB6 154.4 mm to (38.7, 68.6)
- moved C48 151.6 mm to (45.1, 75.6), turned to 180 degrees
- moved U3 147.3 mm to (45.7, 80.6), turned to 0 degrees
- moved NB10 139.1 mm to (51.4, 76.8), turned to 0 degrees
- moved RV4 125.7 mm to (46.4, 71.2)
- moved R23 125.3 mm to (31.1, 64.1), turned to 180 degrees
- moved C22 125.1 mm to (39.4, 43.2), turned to 270 degrees
- moved U2 122.7 mm to (36.2, 48.9)
- moved C5 120.6 mm to (3.17, 61.0), turned to 90 degrees
- moved RV3 119.8 mm to (66.7, 71.2)
- moved R9 119.4 mm to (64.8, 80.6), turned to 0 degrees
- moved C7 117.7 mm to (56.5, 80.6), turned to 90 degrees
- moved R14 116.3 mm to (64.8, 74.3), turned to 180 degrees
- moved U6 116.3 mm to (31.1, 57.8), turned to 180 degrees
- moved Q2 115.2 mm to (73.0, 80.6), turned to 180 degrees
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Connections:
- net Net-(U8-Pad1) renamed /MISO
- net Net-(U8-Pad3) renamed /SCK
- net Net-(U8-Pad4) renamed /MOSI
- C18 pad 1: Net-(C18-Pad1) -> /FV_LOUT
- C20 pad 1: Net-(C20-Pad1) -> /TONE_OUT
- C23 pad 1: Net-(C23-Pad1) -> /FV_ROUT
- C24 pad 1: Net-(C24-Pad1) -> /TONE_OUT
- J3 pad 1: Net-(J3-Pad1) -> (no net)
- J4 pad 1: Net-(J4-Pad1) -> (no net)
- J5 pad 1: Net-(J5-Pad1) -> (no net)
- J6 pad 1: Net-(J6-Pad1) -> (no net)
- R25 pad 2: Net-(NB9-Pad2) -> Net-(R25-Pad2)
- R28 pad 2: Net-(NB9-Pad2) -> Net-(R25-Pad2)
- R30 pad 2: Net-(NB14-Pad2) -> Net-(R30-Pad2)
- R32 pad 2: Net-(NB14-Pad2) -> Net-(R30-Pad2)
- RV8 pad 1: Net-(NB9-Pad2) -> Net-(R25-Pad2)
- RV8 pad 4: Net-(NB14-Pad2) -> Net-(R30-Pad2)
- U11 pad 13: Net-(U11-Pad13) -> (no net)
- U11 pad 5: Net-(U11-Pad5) -> (no net)
- U11 pad 6: Net-(U11-Pad6) -> (no net)
- U2 pad 1: Net-(NB8-Pad2) -> LOUT
- U2 pad 2: Net-(NB9-Pad1) -> Net-(R25-Pad2)
- U2 pad 6: Net-(NB14-Pad1) -> Net-(R30-Pad2)
- U2 pad 7: Net-(NB13-Pad2) -> ROUT
- U9 pad 1: Net-(U9-Pad1) -> /LED_CK
- U9 pad 12: /LED_RST -> (no net)
- U9 pad 13: /LED_CK -> (no net)
- U9 pad 14: /LED_DT -> (no net)
- U9 pad 19: Net-(U9-Pad19) -> (no net)
- U9 pad 2: Net-(U9-Pad2) -> /LED_DT
- U9 pad 22: Net-(U9-Pad22) -> (no net)
- U9 pad 32: Net-(U9-Pad32) -> /LED_RST
Routing:
- net GND: track 0.00 -> 92.2 mm, vias 0 -> 6
- net VDD: track 0.00 -> 41.9 mm, vias 0 -> 3
- net +3V3: track 0.00 -> 31.0 mm, vias 0 -> 7
- net Net-(D2-Pad2): track 0.00 -> 25.8 mm
- net Net-(C16-Pad1): track 0.00 -> 22.0 mm
- net VGND: track 0.00 -> 22.0 mm
- net Net-(C39-Pad1): track 0.00 -> 20.9 mm
- net Net-(C45-Pad1): track 0.00 -> 20.6 mm
- net /SCK: track 0.00 -> 17.4 mm
- net Net-(C4-Pad1): track 0.00 -> 16.0 mm
- net Net-(C33-Pad2): track 0.00 -> 14.1 mm
- net Net-(C43-Pad1): track 0.00 -> 14.1 mm
- net Net-(C35-Pad1): track 0.00 -> 14.0 mm
- net Net-(C38-Pad2): track 0.00 -> 14.0 mm
- net Net-(C40-Pad1): track 0.00 -> 13.3 mm
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- added copper zone on In2.Cu, net +3V3
- added copper zone on B.Cu, net GND
- added copper zone on In2.Cu, net VDD
Other:
- board text added: "3V3"
- board text added: "GND"
- board text added: "Red Myst"
- board text added: "TX"
- board text added: "program"

Commit message: routing continued...
Parts:
- moved R30 19.6 mm to (43.8, 54.6), turned to 0 degrees
- moved C25 18.7 mm to (1.27, 13.3)
- moved NB2 18.5 mm to (39.4, 86.4), turned to 270 degrees
- moved C34 18.5 mm to (16.5, 8.89), turned to 180 degrees
- moved R21 17.0 mm to (9.53, 24.8), turned to 270 degrees
- moved R32 16.3 mm to (43.8, 52.1), turned to 0 degrees
- moved C26 15.3 mm to (21.6, 21.6), turned to 270 degrees
- moved J2 13.7 mm to (16.1, 23.5), turned to 180 degrees
- moved NB6 12.0 mm to (42.5, 80.0), turned to 270 degrees
- moved Y2 6.19 mm to (16.5, 15.9), turned to 90 degrees
- moved R19 5.99 mm to (1.91, 24.8), turned to 270 degrees
- moved R20 5.99 mm to (4.45, 24.8), turned to 90 degrees
- moved R22 5.99 mm to (6.99, 24.8), turned to 270 degrees
- moved U9 4.49 mm to (8.26, 14.0)
- moved R25 2.54 mm to (33.0, 43.2)
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Connections:
- U9 pad 23: /S0 -> /S2
- U9 pad 25: /S2 -> /S0
Routing:
- net VGND: track 22.0 -> 121.6 mm
- net /WP: track 0.00 -> 58.3 mm
- net /SCL: track 0.00 -> 55.4 mm
- net Net-(C10-Pad1): track 0.00 -> 50.9 mm
- net /SDA: track 0.00 -> 49.0 mm, vias 0 -> 1
- net LOUT: track 0.00 -> 48.3 mm
- net /S2: track 0.00 -> 48.2 mm
- net /S1: track 0.00 -> 46.0 mm
- net +3V3: track 31.0 -> 75.6 mm, vias 7 -> 10
- net /S0: track 0.00 -> 44.1 mm
- net GND: track 92.2 -> 129.8 mm, vias 6 -> 15
- net Net-(R29-Pad2): track 0.00 -> 33.3 mm
- net Net-(R27-Pad2): track 0.00 -> 32.0 mm
- net ROUT: track 0.00 -> 26.3 mm
- net Net-(R24-Pad2): track 0.00 -> 21.6 mm
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
Commit message: routing done
Parts:
- moved RN3 6.38 mm to (59.1, 19.7)
- moved RN4 5.12 mm to (52.1, 19.7)
- moved RN1 4.49 mm to (44.5, 19.7)
- moved RN2 4.49 mm to (38.7, 19.7)
- moved U10 1.91 mm to (45.1, 27.3)
Connections:
- J3 pad 1: (no net) -> Net-(J3-Pad1)
- J4 pad 1: (no net) -> Net-(J4-Pad1)
- J5 pad 1: (no net) -> Net-(J5-Pad1)
- J6 pad 1: (no net) -> Net-(J6-Pad1)
- SS1 pad 1: Net-(RN1-Pad8) -> Net-(RN2-Pad7)
- SS1 pad 2: Net-(RN1-Pad7) -> Net-(RN2-Pad5)
- SS1 pad 4: Net-(RN1-Pad6) -> Net-(RN1-Pad7)
- SS1 pad 6: Net-(RN2-Pad5) -> Net-(RN1-Pad6)
- SS1 pad 7: Net-(RN2-Pad6) -> Net-(RN1-Pad8)
- SS1 pad 9: Net-(RN2-Pad7) -> Net-(RN2-Pad6)
- SS2 pad 1: Net-(RN3-Pad8) -> Net-(RN4-Pad7)
- SS2 pad 2: Net-(RN3-Pad7) -> Net-(RN4-Pad5)
- SS2 pad 4: Net-(RN3-Pad6) -> Net-(RN3-Pad7)
- SS2 pad 6: Net-(RN4-Pad5) -> Net-(RN3-Pad6)
- SS2 pad 7: Net-(RN4-Pad6) -> Net-(RN3-Pad8)
- SS2 pad 9: Net-(RN4-Pad7) -> Net-(RN4-Pad6)
- SW1 pad 4: Net-(SW1-Pad4) -> /ROT_SW
- U11 pad 13: (no net) -> Net-(U11-Pad13)
- U11 pad 5: (no net) -> Net-(U11-Pad5)
- U11 pad 6: (no net) -> Net-(U11-Pad6)
- U9 pad 11: Net-(SW1-Pad3) -> /ROT_SW
- U9 pad 12: (no net) -> Net-(U9-Pad12)
- U9 pad 13: (no net) -> Net-(U9-Pad13)
- U9 pad 14: (no net) -> Net-(U9-Pad14)
- U9 pad 19: (no net) -> Net-(U9-Pad19)
- U9 pad 2: /LED_DT -> /LED_RST
- U9 pad 22: (no net) -> Net-(U9-Pad22)
- U9 pad 32: /LED_RST -> /LED_DT
- U9 pad 9: Net-(SW1-Pad4) -> Net-(SW1-Pad3)
Routing:
- net Net-(RV2-Pad2): track 0.00 -> 82.8 mm, vias 0 -> 1
- net Net-(RV3-Pad2): track 0.00 -> 60.5 mm, vias 0 -> 1
- net /TONE_OUT: track 2.54 -> 62.7 mm, vias 0 -> 3
- net /T0: track 6.00 -> 53.6 mm, vias 0 -> 2
- net /LED_RST: track 0.00 -> 46.0 mm, vias 0 -> 2
- net /LED_CK: track 0.00 -> 45.2 mm, vias 0 -> 2
- net Net-(RV4-Pad2): track 0.00 -> 38.1 mm, vias 0 -> 1
- net +3V3: track 75.6 -> 112.0 mm, vias 10 -> 11
- net Net-(RN2-Pad1): track 0.00 -> 28.3 mm, vias 0 -> 2
- net Net-(SW1-Pad1): track 0.00 -> 27.4 mm
- net /LED_DT: track 0.00 -> 24.3 mm
- net Net-(SW1-Pad3): track 0.00 -> 23.9 mm
- net Net-(R31-Pad2): track 18.2 -> 41.1 mm, vias 0 -> 1
- net Net-(RN3-Pad1): track 0.00 -> 20.9 mm
- net Net-(RN3-Pad2): track 0.00 -> 20.4 mm
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Other:
- rule trace_min: 0.2 -> 0.2032
- board text added: "Green Myst"
- board text removed: "Red Myst"
