File: circuit/RedMyst.kicad_pcb (KiCad board)
At the start: 4 copper layers, 100 x 100 mm, 146 parts, among them J1 JACK_MONO, J2 CONN_01X03, J3 HOLE, J4 HOLE, J5 HOLE, J6 HOLE, J7 Barrel_Jack_Switch, Q1 MMBFJ201, Q2 BC547, Q3 BC557, SW1 ROT_SW, SW2 ON/OFF, U1 NE5532, U10 74164, U11 TPA3136D2, U2 NE5532, U3 TLE2426, U4 FV-1, U5 LM1117, U6 24LC32A, U7 74164, U8 AVR-ISP6, U9 ATMEGA8, Y1 32768Hz, Y2 8MHz

Commit message: final touches
Parts:
- moved R33 0.64 mm to (17.8, 3.81)
- moved RN1 0.63 mm to (45.1, 19.7)
Routing:
- net VDD: track 51.0 -> 59.5 mm, vias 5 -> 7
- net Net-(RN1-Pad8): track 19.4 -> 18.1 mm
- net Net-(RN1-Pad5): track 4.06 -> 2.82 mm
- net Net-(RN1-Pad6): track 19.2 -> 18.4 mm
- net Net-(RN1-Pad1): track 16.8 -> 17.6 mm
- net Net-(RN1-Pad3): track 16.5 -> 17.3 mm
- net Net-(RN1-Pad4): track 16.2 -> 16.9 mm
- net +3V3: track 112.0 -> 111.3 mm
- net Net-(SW1-Pad1): track 27.4 -> 28.1 mm
- net Net-(RN1-Pad2): track 17.1 -> 17.7 mm
- net Net-(C45-Pad1): track 20.6 -> 21.2 mm
- net Net-(RN2-Pad1): track 28.3 -> 28.9 mm
- net Net-(C45-Pad2): track 11.4 -> 12.0 mm
- added copper zone on In1.Cu, net GND

Commit message: and continued...
Parts:
- moved C42 0.64 mm to (78.1, 32.4)
- moved C40 0.64 mm to (78.1, 26.0)
