File: circuit/modulo.kicad_pcb (KiCad board)
At the start: 4 copper layers, 100 x 50 mm, 139 parts, among them J1 JACK_MONO, J2 CONN_01X03, J3 HOLE, J4 Barrel_Jack_Switch, J5 HOLE, J6 HOLE, J7 HOLE, Q1 MMBFJ201, Q2 BC547, Q3 BC557, SW1 ROT_SW, SW2 ON/OFF, U1 TLE2426, U10 ATMEGA8, U11 74164, U12 TPA3136D2, U2 NE5532, U3 FV-1, U4 NE5532, U5 24LC32A, U6 NE5532, U7 LM1117, U8 74164, U9 AVR-ISP6, Y1 32768Hz, Y2 8MHz

Commit message: started routing the preamp
Parts:
- C22, C23: footprint myAmp:C_1206 -> myAmp:C_5MM_1206
- RV1, RV2: footprint myAmp:ALPS_RK09L -> myAmp:BOURNS_PTD901_xx15K
- RV3: renamed from RV6; footprint myAmp:ALPS_RK09L -> myAmp:BOURNS_PTD901_xx15K
- moved Q1 202.6 mm to (37.0, 32.0)
- moved C16 198.5 mm to (32.4, 62.2), turned to 90 degrees
- moved C1 191.0 mm to (44.5, 32.4), turned to 270 degrees
- moved R15 186.0 mm to (22.9, 64.8), turned to 180 degrees
- moved J5 185.8 mm to (4.00, 46.0)
- moved R25 181.9 mm to (22.9, 57.1)
- moved R7 179.1 mm to (30.5, 32.4), turned to 90 degrees
- moved Q2 177.4 mm to (14.0, 62.2), turned to 90 degrees
- moved C20 174.8 mm to (32.4, 54.6), turned to 90 degrees
- moved U1 172.8 mm to (39.4, 58.4), turned to 270 degrees
- moved Q3 164.3 mm to (14.0, 54.6), turned to 270 degrees
- moved R27 160.6 mm to (22.9, 52.1)
- moved C3 158.5 mm to (41.3, 52.7), turned to 180 degrees
- moved C10 157.2 mm to (72.4, 27.9)
- moved C22 153.8 mm to (54.6, 34.3)
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- renumbered RV3 to RV4, RV4 to RV5, RV5 to RV6
Connections:
- C16 pad 2: VGND -> /PA_VGND
- C20 pad 1: VGND -> /PA_VGND
- C3 pad 2: VGND -> /PA_VGND
- C4 pad 2: (no net) -> /FV_LIN
- C42 pad 2: (no net) -> Net-(C42-Pad2)
- C45 pad 2: (no net) -> Net-(C45-Pad2)
- C47 pad 2: (no net) -> Net-(C47-Pad2)
- C48 pad 2: (no net) -> Net-(C48-Pad2)
- C49 pad 2: (no net) -> /FV_RIN
- D4 pad 1: VGND -> /PA_VGND
- D5 pad 2: VGND -> /PA_VGND
- J3 pad 1: (no net) -> Net-(J3-Pad1)
- J5 pad 1: (no net) -> Net-(J5-Pad1)
- J6 pad 1: (no net) -> Net-(J6-Pad1)
- J7 pad 1: (no net) -> Net-(J7-Pad1)
- R10 pad 1: VGND -> /PA_VGND
- R13 pad 2: VGND -> /PA_VGND
- R22 pad 1: VGND -> /PA_VGND
- R25 pad 2: VGND -> /PA_VGND
- R5 pad 2: VGND -> /PA_VGND
- RV3 pad 1: VGND -> /PA_VGND
- U1 pad 1: VGND -> /PA_VGND
- U10 pad 12: (no net) -> Net-(U10-Pad12)
- U10 pad 13: (no net) -> Net-(U10-Pad13)
- U10 pad 14: (no net) -> Net-(U10-Pad14)
- U10 pad 19: (no net) -> Net-(U10-Pad19)
- U10 pad 22: (no net) -> Net-(U10-Pad22)
- U12 pad 13: (no net) -> Net-(U12-Pad13)
- U12 pad 5: (no net) -> Net-(U12-Pad5)
- U12 pad 6: (no net) -> Net-(U12-Pad6)
Other:
- outline, holes or cut-outs redrawn

Commit message: preamp layout started
Parts:
- added R2: 1, myAmp:R_10MM, F.Cu at (34.9, 14.0)
- added R37: 1M, myAmp:R_10MM, F.Cu at (33.7, 29.2)
- added R38: 100, myAmp:R_10MM, F.Cu at (33.7, 31.9)
- added R9: 1, myAmp:R_10MM, F.Cu at (45.1, 14.0)
- added SW3: Idss/Vp, myAmp:PIN_1x03, F.Cu at (31.7, 35.6)
- added SW4: disc/TLE2426, myAmp:ESP2010_switch, F.Cu at (85.7, 2.54)
- added TPoint1: CONN_01X02, myAmp:TestPoints, F.Cu at (38.7, 25.4)
- added TPow1: TestDC, myAmp:TestPower, F.Cu at (33.0, 25.4)
- added U13: modulo-bus, myAmp:modulo-bus, F.Cu at (75.3, -26.4)
- added U14: modulo-bus, myAmp:modulo-bus, F.Cu at (45.7, 1.91)
- C10, C7: footprint myAmp:C_1206 -> myAmp:C_5MM_1206
- Q1: footprint myAmp:SOT-23 -> myAmp:SOT-23_with_jig
- moved C25 168.8 mm to (67.9, -12.7)
- moved D7 137.4 mm to (91.8, -14.1)
- moved D1 134.5 mm to (16.5, 34.3)
- moved C7 129.8 mm to (61.0, 14.6), turned to 270 degrees
- moved C9 129.3 mm to (107.0, 8.00)
- moved SW2 112.5 mm to (83.7, -16.8)
- moved R33 111.8 mm to (71.7, -23.2)
- moved D2 110.0 mm to (16.5, 31.1)
- moved U7 102.7 mm to (93.9, -20.6)
- moved Q2 84.2 mm to (94.6, 38.1), turned to 180 degrees
- moved R15 82.4 mm to (97.2, 29.2), turned to 90 degrees
- moved J4 82.3 mm to (59.5, -19.5)
- moved D4 79.6 mm to (94.6, 29.2), turned to 270 degrees
- moved R22 75.6 mm to (92.1, 29.2), turned to 90 degrees
- moved C16 75.4 mm to (94.6, 19.7), turned to 180 degrees
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- renumbered R2 to R39, R9 to R40
Connections:
- net Net-(C1-Pad2) renamed /pre amp/jfet_d
- net Net-(D1-Pad2) renamed /pre amp/jfet_g
- net Net-(Q1-Pad2) renamed /pre amp/jfet_s
- C10 pad 1: /PREAMP_OUT -> Net-(C10-Pad1)
- C16 pad 1: VDD -> +12V
- C16 pad 2: /PA_VGND -> /pre amp/vgnd_disc
- C2 pad 2: Net-(C2-Pad2) -> Net-(C10-Pad1)
- C20 pad 1: /PA_VGND -> /pre amp/vgnd_disc
- C22 pad 2: VDD -> +12V
- C3 pad 2: /PA_VGND -> /pre amp/vgnd_tle
- C4 pad 2: /FV_LIN -> (no net)
- C42 pad 2: Net-(C42-Pad2) -> (no net)
- C45 pad 2: Net-(C45-Pad2) -> (no net)
- C47 pad 2: Net-(C47-Pad2) -> (no net)
- C48 pad 2: Net-(C48-Pad2) -> (no net)
- C49 pad 2: /FV_RIN -> (no net)
- C7 pad 1: Net-(C2-Pad2) -> /pre amp/PREAMP_OUT
- D4 pad 1: /PA_VGND -> /pre amp/vgnd_disc
- D5 pad 2: /PA_VGND -> /pre amp/vgnd_disc
- J3 pad 1: Net-(J3-Pad1) -> (no net)
- J5 pad 1: Net-(J5-Pad1) -> (no net)
- J6 pad 1: Net-(J6-Pad1) -> (no net)
- J7 pad 1: Net-(J7-Pad1) -> (no net)
- Q2 pad 1: VDD -> +12V
- R1 pad 2: VDD -> +12V
- R10 pad 1: /PA_VGND -> /pre amp/PA_VGND
- R10 pad 2: Net-(C7-Pad2) -> Net-(C10-Pad2)
- R11 pad 1: Net-(C7-Pad2) -> Net-(C10-Pad2)
- R11 pad 2: Net-(C2-Pad2) -> Net-(C10-Pad1)
- R12 pad 1: Net-(C10-Pad2) -> Net-(C7-Pad2)
- R12 pad 2: /PREAMP_OUT -> /pre amp/PREAMP_OUT
- R13 pad 1: Net-(C10-Pad2) -> Net-(C7-Pad2)
- R13 pad 2: /PA_VGND -> /pre amp/PA_VGND
- R15 pad 2: VDD -> +12V
- R22 pad 1: /PA_VGND -> /pre amp/vgnd_disc
- R25 pad 2: /PA_VGND -> /pre amp/vgnd_disc
- R4 pad 2: Net-(C2-Pad2) -> Net-(C10-Pad1)
- R5 pad 2: /PA_VGND -> /pre amp/PA_VGND
- RV3 pad 1: /PA_VGND -> /pre amp/PA_VGND
- U1 pad 1: /PA_VGND -> /pre amp/vgnd_tle
- U1 pad 3: VDD -> +12V
- U10 pad 12: Net-(U10-Pad12) -> (no net)
- U10 pad 13: Net-(U10-Pad13) -> (no net)
- U10 pad 14: Net-(U10-Pad14) -> (no net)
- U10 pad 19: Net-(U10-Pad19) -> (no net)
- U10 pad 22: Net-(U10-Pad22) -> (no net)
- U12 pad 13: Net-(U12-Pad13) -> (no net)
- U12 pad 5: Net-(U12-Pad5) -> (no net)
- U12 pad 6: Net-(U12-Pad6) -> (no net)
- U2 pad 1: Net-(C2-Pad2) -> Net-(C10-Pad1)
- U2 pad 2: Net-(C7-Pad2) -> Net-(C10-Pad2)
- U2 pad 6: Net-(C10-Pad2) -> Net-(C7-Pad2)
- U2 pad 7: /PREAMP_OUT -> /pre amp/PREAMP_OUT
- U2 pad 8: VDD -> +12V
Other:
- board text added: "test jig"

Commit message: fully modularized!
Parts:
- added J10: HOLE, myAmp:MountingHole, F.Cu at (197.0, 4.00)
- added J11: HOLE, myAmp:MountingHole, F.Cu at (197.0, 46.0)
- added J12: HOLE, myAmp:MountingHole, F.Cu at (206.0, 4.00)
- added J13: HOLE, myAmp:MountingHole, F.Cu at (206.0, 46.0)
- added J14: HOLE, myAmp:MountingHole, F.Cu at (298.0, 4.00)
- added J15: HOLE, myAmp:MountingHole, F.Cu at (298.0, 46.0)
- added J16: HOLE, myAmp:MountingHole, F.Cu at (298.0, 55.0)
- added J17: HOLE, myAmp:MountingHole, F.Cu at (206.0, 97.0)
- added J18: HOLE, myAmp:MountingHole, F.Cu at (206.0, 55.0)
- added J19: HOLE, myAmp:MountingHole, F.Cu at (298.0, 97.0)
- added J20: HOLE, myAmp:MountingHole, F.Cu at (105.0, 55.0)
- added J21: HOLE, myAmp:MountingHole, F.Cu at (105.0, 97.0)
- added J22: HOLE, myAmp:MountingHole, F.Cu at (197.0, 55.0)
- added J23: HOLE, myAmp:MountingHole, F.Cu at (197.0, 97.0)
- added J24: HOLE, myAmp:MountingHole, F.Cu at (4.00, 55.0)
- added J25: HOLE, myAmp:MountingHole, F.Cu at (4.00, 97.0)
- added J26: HOLE, myAmp:MountingHole, F.Cu at (96.0, 55.0)
- added J27: HOLE, myAmp:MountingHole, F.Cu at (96.0, 97.0)
- added J8: HOLE, myAmp:MountingHole, F.Cu at (105.0, 4.00)
- added J9: HOLE, myAmp:MountingHole, F.Cu at (105.0, 46.3)
- C11, C14: value 1µF -> 1nF
- C13, C15: value 100nF -> 1µF
- C17: value 15pF -> 100nF
- C23: value 100nF -> 1µF; footprint myAmp:C_5MM_1206 -> myAmp:C_1206
- C24: value 1µF -> 100nF; footprint myAmp:C_1206 -> myAmp:C_5MM_1206
- C26: value 100nF -> 22pF
- C29: value 100nF -> 1μF
- C30, C33: value 1nF -> 1μF
- C31: value 100μF -> 1μF; footprint myAmp:CPOL_D8_P3.5 -> myAmp:C_1206
- C34, C36: value 680nF -> 1μF; footprint myAmp:C_FILM_5MM -> myAmp:C_1206
- C35: value 22pF -> 100nF
- C37: value 1μF -> 1nF
- C38: value 1μF -> 100μF; footprint myAmp:C_1206 -> myAmp:CPOL_D8_P3.5
- C39: value 680nF -> 100nF; footprint myAmp:C_FILM_5MM -> myAmp:C_1206
- C4: value 1µF -> 15pF
- C40: value 220nF -> 1nF
- C42: value 1μF -> 220nF
- C44: value 680nF -> 220nF; footprint myAmp:C_FILM_5MM -> myAmp:C_1206
- C45, C47, C48: value 1μF -> 680nF; footprint myAmp:C_1206 -> myAmp:C_FILM_5MM
- C46: value 220nF -> 680nF; footprint myAmp:C_1206 -> myAmp:C_FILM_5MM
- C49: value 1µF -> 10nF
- C5, C6: value 10nF -> 1µF
- C50: value 1nF -> 10nF
- C9: value 1nF -> 100nF
- R14: value 100 -> 1K
- R20: value 10K -> 100
- R26: value 10K -> 1K
- R3: value 1K -> 100
- R34: value 2K2 -> 10K
- R35: value 10K -> 2K2
- R39: value 1K -> 10K
- R40: value 100 -> 10K
- U10: value ATMEGA8 -> 74164; footprint myAmp:TQFP-32_7x7mm_Pitch0.8mm -> myAmp:SOIC-14_3.9x8.7mm_P1.27mm
- U8: value 74164 -> ATMEGA8; footprint myAmp:SOIC-14_3.9x8.7mm_P1.27mm -> myAmp:TQFP-32_7x7mm_Pitch0.8mm
- moved C18 191.0 mm to (44.2, 84.4)
- moved U6 188.4 mm to (60.5, 69.2)
- moved C23 187.4 mm to (56.9, 81.7)
- moved R24 178.0 mm to (34.9, 78.9)
- moved U4 170.4 mm to (68.9, 69.2)
- moved R28 164.1 mm to (47.6, 81.6)
- moved C21 161.2 mm to (50.0, 84.4)
- moved C9 159.5 mm to (263.6, 38.7)
- moved R23 157.5 mm to (60.4, 78.9)
- moved C19 154.4 mm to (69.7, 73.8)
- moved RV4 147.2 mm to (262.6, 22.0)
- moved R30 144.7 mm to (34.9, 84.3)
- moved R16 141.7 mm to (276.0, 21.2)
- moved R21 141.0 mm to (276.0, 13.0)
- moved R14 139.9 mm to (262.1, 27.5)
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Connections:
- C11 pad 1: Net-(C11-Pad1) -> GND
- C11 pad 2: GND -> Net-(C11-Pad2)
- C13 pad 1: +3V3 -> GND
- C13 pad 2: GND -> /FV-1/MID
- C14 pad 2: /MID -> Net-(C14-Pad2)
- C15 pad 1: GND -> Net-(C15-Pad1)
- C15 pad 2: +3V3 -> GND
- C17 pad 1: Net-(C17-Pad1) -> +3V3
- C18 pad 1: /FV_LOUT -> /mixer/FV_LOUT
- C19 pad 1: /TONE_OUT -> /mixer/TONE_OUT
- C21 pad 1: /FV_ROUT -> /mixer/FV_ROUT
- C23 pad 1: GND -> /mixer/TONE_OUT
- C23 pad 2: VDD -> Net-(C23-Pad2)
- C24 pad 1: /TONE_OUT -> GND
- C24 pad 2: Net-(C24-Pad2) -> VDD
- C26 pad 1: GND -> Net-(C26-Pad1)
- C26 pad 2: +3V3 -> GND
- C30 pad 1: VDD -> Net-(C30-Pad1)
- C30 pad 2: GND -> Net-(C30-Pad2)
- C31 pad 1: VDD -> Net-(C31-Pad1)
- C31 pad 2: GND -> Net-(C31-Pad2)
- C33 pad 1: VDD -> /Class D audio power amp/GVDD
- C34 pad 1: GND -> Net-(C34-Pad1)
- C35 pad 1: Net-(C35-Pad1) -> GND
- C35 pad 2: GND -> +3V3
- C36 pad 2: GND -> Net-(C36-Pad2)
- C38 pad 1: /GVDD -> VDD
- C39 pad 1: GND -> VDD
- C39 pad 2: Net-(C39-Pad2) -> GND
- C4 pad 2: (no net) -> GND
- C40 pad 1: Net-(C40-Pad1) -> VDD
- C40 pad 2: Net-(C40-Pad2) -> GND
- C42 pad 2: (no net) -> Net-(C42-Pad2)
- C44 pad 2: GND -> Net-(C44-Pad2)
- C45 pad 1: Net-(C45-Pad1) -> GND
- C45 pad 2: (no net) -> Net-(C45-Pad2)
- C46 pad 2: Net-(C46-Pad2) -> GND
- C47 pad 1: Net-(C47-Pad1) -> GND
- C47 pad 2: (no net) -> Net-(C47-Pad2)
- C48 pad 2: (no net) -> GND
- C49 pad 1: Net-(C49-Pad1) -> /FV-1/FV_LOUT
- C49 pad 2: (no net) -> GND
- C5 pad 1: /FV_LOUT -> Net-(C5-Pad1)
- C5 pad 2: GND -> /FV-1/FV_RIN
- C50 pad 1: GND -> /FV-1/FV_ROUT
- C50 pad 2: Net-(C50-Pad2) -> GND
- C6 pad 1: /FV_ROUT -> Net-(C6-Pad1)
- C6 pad 2: GND -> /FV-1/FV_LIN
- C9 pad 2: Net-(C9-Pad2) -> +3V3
- J2 pad 3: /DBG_TX -> /mcu/DBG_TX
- J3 pad 1: (no net) -> Net-(J3-Pad1)
- J5 pad 1: (no net) -> Net-(J5-Pad1)
- J6 pad 1: (no net) -> Net-(J6-Pad1)
- J7 pad 1: (no net) -> Net-(J7-Pad1)
- L1 pad 1: Net-(C40-Pad1) -> Net-(C41-Pad1)
- L1 pad 2: Net-(C34-Pad2) -> Net-(C45-Pad2)
- L2 pad 1: Net-(C41-Pad1) -> Net-(C42-Pad1)
- L2 pad 2: Net-(C36-Pad1) -> Net-(C46-Pad1)
- L3 pad 2: Net-(C39-Pad2) -> Net-(C47-Pad2)
- L4 pad 1: Net-(C46-Pad1) -> Net-(C44-Pad1)
- L4 pad 2: Net-(C44-Pad1) -> Net-(C48-Pad1)
- R14 pad 1: Net-(D3-Pad1) -> Net-(C6-Pad1)
- R14 pad 2: Net-(R14-Pad2) -> Net-(C14-Pad2)
- R16 pad 1: /S2 -> /FV-1/T0
- R16 pad 2: GND -> +3V3
- R18 pad 1: Net-(R17-Pad2) -> Net-(C19-Pad2)
- R19 pad 1: GND -> /FV-1/WP
- R19 pad 2: /S1 -> +3V3
- R20 pad 1: /T0 -> +3V3
- R20 pad 2: +3V3 -> Net-(C15-Pad1)
- R21 pad 1: /S0 -> /FV-1/S0
- R23 pad 1: Net-(C19-Pad2) -> Net-(C21-Pad2)
- R24 pad 1: Net-(R23-Pad2) -> Net-(C23-Pad2)
- R24 pad 2: Net-(R18-Pad2) -> Net-(R24-Pad2)
- R26 pad 1: /WP -> /FV-1/FV_LOUT
- R26 pad 2: +3V3 -> Net-(R26-Pad2)
- R28 pad 1: Net-(C21-Pad2) -> Net-(R17-Pad2)
- R29 pad 1: Net-(R28-Pad2) -> Net-(R18-Pad2)
- R29 pad 2: Net-(R29-Pad2) -> Net-(R28-Pad2)
- R3 pad 1: /FV_ROUT -> Net-(D3-Pad1)
- R30 pad 1: Net-(C24-Pad2) -> Net-(R23-Pad2)
- R31 pad 1: Net-(R30-Pad2) -> Net-(R24-Pad2)
- R31 pad 2: Net-(R29-Pad2) -> Net-(R30-Pad2)
- R32 pad 1: /AVR_RST -> /mcu/AVR_RST
- R34 pad 1: /SD_FAULT -> VDD
- R34 pad 2: Net-(D6-Pad1) -> /Class D audio power amp/SD_FAULT
- R35 pad 1: VDD -> /Class D audio power amp/SD_FAULT
- R35 pad 2: /SD_FAULT -> Net-(D6-Pad1)
- R36 pad 1: Net-(C49-Pad1) -> /FV-1/FV_ROUT
- R36 pad 2: Net-(C50-Pad2) -> Net-(R36-Pad2)
- R39 pad 1: /FV_LOUT -> GND
- R39 pad 2: Net-(R39-Pad2) -> /FV-1/S1
- R40 pad 1: +3V3 -> /FV-1/S2
- R40 pad 2: Net-(C11-Pad1) -> GND
- R6 pad 1: Net-(C4-Pad1) -> Net-(C5-Pad1)
- R6 pad 2: Net-(C9-Pad2) -> Net-(C11-Pad2)
- RV7 pad 3: Net-(R23-Pad2) -> Net-(R18-Pad2)
- RV7 pad 4: Net-(R18-Pad2) -> Net-(R23-Pad2)
- RV7 pad 5: LOUT -> VGND
- RV7 pad 6: LOUT -> Net-(R24-Pad2)
- RV8 pad 2: VGND -> LOUT
- RV8 pad 3: Net-(R30-Pad2) -> LOUT
- RV8 pad 4: Net-(R29-Pad2) -> Net-(R30-Pad2)
- S1 pad 1: Net-(C34-Pad2) -> Net-(C45-Pad2)
- S1 pad 2: Net-(C36-Pad1) -> Net-(C46-Pad1)
- S2 pad 1: Net-(C39-Pad2) -> Net-(C47-Pad2)
- S2 pad 2: Net-(C44-Pad1) -> Net-(C48-Pad1)
- SW1 pad 4: /ROT_SW -> /mcu/ROT_SW
- U10 pad 1: /LED_CK -> /mcu/LED_DT
- U10 pad 10: Net-(SW1-Pad1) -> Net-(RN2-Pad4)
- U10 pad 11: /ROT_SW -> Net-(RN2-Pad3)
- U10 pad 12: (no net) -> Net-(RN2-Pad2)
- U10 pad 13: (no net) -> Net-(RN2-Pad1)
- U10 pad 14: (no net) -> +3V3
- U10 pad 2: /LED_RST -> /mcu/LED_DT
- U10 pad 3: GND -> Net-(RN1-Pad1)
- U10 pad 4: +3V3 -> Net-(RN1-Pad2)
- U10 pad 5: GND -> Net-(RN1-Pad3)
- U10 pad 6: +3V3 -> Net-(RN1-Pad4)
- U10 pad 7: Net-(C27-Pad1) -> GND
- U10 pad 8: Net-(C35-Pad1) -> /mcu/LED_CK
- U10 pad 9: Net-(SW1-Pad3) -> /mcu/LED_RST
- U11 pad 8: /LED_CK -> /mcu/LED_CK
- U11 pad 9: /LED_RST -> /mcu/LED_RST
- U12 pad 1: /SD_FAULT -> /Class D audio power amp/SD_FAULT
- U12 pad 10: /GVDD -> /Class D audio power amp/GVDD
- U12 pad 11: Net-(C47-Pad1) -> Net-(C36-Pad1)
- U12 pad 12: Net-(C48-Pad1) -> Net-(C31-Pad1)
- U12 pad 13: (no net) -> Net-(U12-Pad13)
- U12 pad 17: Net-(C46-Pad2) -> Net-(C44-Pad2)
- U12 pad 18: Net-(C46-Pad1) -> Net-(C44-Pad1)
- U12 pad 2: /SD_FAULT -> /Class D audio power amp/SD_FAULT
- U12 pad 22: Net-(C41-Pad2) -> Net-(C42-Pad2)
- U12 pad 23: Net-(C41-Pad1) -> Net-(C42-Pad1)
- U12 pad 25: Net-(C40-Pad1) -> Net-(C41-Pad1)
- U12 pad 26: Net-(C40-Pad2) -> Net-(C41-Pad2)
- U12 pad 3: Net-(C42-Pad1) -> Net-(C34-Pad1)
- U12 pad 4: Net-(C45-Pad1) -> Net-(C30-Pad1)
- U12 pad 5: (no net) -> Net-(U12-Pad5)
- U12 pad 6: (no net) -> Net-(U12-Pad6)
- U12 pad 9: /GVDD -> /Class D audio power amp/GVDD
- U13 pad 1: (no net) -> Net-(U13-Pad1)
- U13 pad 10: (no net) -> Net-(U13-Pad10)
- U13 pad 11: (no net) -> Net-(U13-Pad11)
- U13 pad 12: (no net) -> Net-(U13-Pad12)
- U13 pad 13: (no net) -> Net-(U13-Pad13)
- U13 pad 14: (no net) -> Net-(U13-Pad14)
- U13 pad 15: (no net) -> Net-(U13-Pad15)
- U13 pad 16: (no net) -> Net-(U13-Pad16)
- U13 pad 17: (no net) -> Net-(U13-Pad17)
- U13 pad 18: (no net) -> Net-(U13-Pad18)
- U13 pad 19: (no net) -> Net-(U13-Pad19)
- U13 pad 2: (no net) -> Net-(U13-Pad2)
- U13 pad 3: (no net) -> Net-(U13-Pad3)
- U13 pad 4: (no net) -> Net-(U13-Pad4)
- U13 pad 5: (no net) -> Net-(U13-Pad5)
- U13 pad 6: (no net) -> Net-(U13-Pad6)
- U13 pad 7: (no net) -> Net-(U13-Pad7)
- U13 pad 8: (no net) -> Net-(U13-Pad8)
- U13 pad 9: (no net) -> Net-(U13-Pad9)
- U14 pad 10: (no net) -> Net-(U14-Pad10)
- U14 pad 11: (no net) -> Net-(U14-Pad11)
- U14 pad 12: (no net) -> Net-(U14-Pad12)
- U14 pad 13: (no net) -> Net-(U14-Pad13)
- U14 pad 14: (no net) -> Net-(U14-Pad14)
- U14 pad 15: (no net) -> Net-(U14-Pad15)
- U14 pad 16: (no net) -> Net-(U14-Pad16)
- U14 pad 17: (no net) -> Net-(U14-Pad17)
- U14 pad 18: (no net) -> Net-(U14-Pad18)
- U14 pad 19: (no net) -> Net-(U14-Pad19)
- U14 pad 2: (no net) -> Net-(U14-Pad2)
- U14 pad 4: (no net) -> Net-(U14-Pad4)
- U14 pad 5: (no net) -> Net-(U14-Pad5)
- U14 pad 8: (no net) -> Net-(U14-Pad8)
- U14 pad 9: (no net) -> Net-(U14-Pad9)
- U3 pad 1: Net-(C9-Pad2) -> Net-(C14-Pad2)
- U3 pad 13: /T0 -> /FV-1/T0
- U3 pad 14: /SCL -> /FV-1/SCL
- U3 pad 15: /SDA -> /FV-1/SDA
- U3 pad 16: /S0 -> /FV-1/S0
- U3 pad 17: /S1 -> /FV-1/S1
- U3 pad 18: /S2 -> /FV-1/S2
- U3 pad 2: Net-(C50-Pad2) -> Net-(C11-Pad2)
- U3 pad 26: Net-(C11-Pad1) -> Net-(C15-Pad1)
- U3 pad 27: Net-(R3-Pad2) -> Net-(R36-Pad2)
- U3 pad 28: Net-(R39-Pad2) -> Net-(R26-Pad2)
- U3 pad 3: /MID -> /FV-1/MID
- U3 pad 5: Net-(R14-Pad2) -> Net-(R3-Pad2)
- U3 pad 9: Net-(C17-Pad1) -> Net-(C4-Pad1)
- U4 pad 2: Net-(R18-Pad2) -> Net-(R28-Pad2)
- U4 pad 6: Net-(R29-Pad2) -> Net-(R30-Pad2)
- U5 pad 5: /SDA -> /FV-1/SDA
- U5 pad 6: /SCL -> /FV-1/SCL
- U5 pad 7: /WP -> /FV-1/WP
- U8 pad 1: /LED_DT -> /mcu/LED_CK
- U8 pad 10: Net-(RN2-Pad4) -> Net-(SW1-Pad1)
- U8 pad 11: Net-(RN2-Pad3) -> /mcu/ROT_SW
- U8 pad 12: Net-(RN2-Pad2) -> Net-(U8-Pad12)
- U8 pad 13: Net-(RN2-Pad1) -> Net-(U8-Pad13)
- U8 pad 14: +3V3 -> Net-(U8-Pad14)
- U8 pad 2: /LED_DT -> /mcu/LED_RST
- U8 pad 3: Net-(RN1-Pad1) -> GND
- U8 pad 4: Net-(RN1-Pad2) -> +3V3
- U8 pad 5: Net-(RN1-Pad3) -> GND
- U8 pad 6: Net-(RN1-Pad4) -> +3V3
- U8 pad 7: GND -> Net-(C26-Pad1)
- U8 pad 8: /LED_CK -> Net-(C27-Pad1)
- U8 pad 9: /LED_RST -> Net-(SW1-Pad3)
- U9 pad 1: /MISO -> /mcu/MISO
- U9 pad 3: /SCK -> /mcu/SCK
- U9 pad 4: /MOSI -> /mcu/MOSI
- U9 pad 5: /AVR_RST -> /mcu/AVR_RST
- Y1 pad 1: Net-(C17-Pad1) -> Net-(C4-Pad1)
- Y2 pad 1: Net-(C27-Pad1) -> Net-(C26-Pad1)
- Y2 pad 2: Net-(C35-Pad1) -> Net-(C27-Pad1)
Other:
- board size 100 x 50 mm -> 302 x 101 mm

Commit message: half way laying out the mixer
Parts:
- added C51: 10µF, myAmp:CPOL_D4_P1.5, F.Cu at (228.0, 27.3)
- added C52: 220μF, myAmp:CPOL_D6.3_P2.5, F.Cu at (51.9, 124.5)
- added C53: 220μF, myAmp:CPOL_D6.3_P2.5, F.Cu at (59.3, 124.5)
- added C54: 100nF, myAmp:C_5MM_1206, F.Cu at (65.0, 115.0)
- added D8: 1N4148, myAmp:DO35, F.Cu at (45.6, 114.0)
- added D9: 1N4148, myAmp:DO35, F.Cu at (55.8, 114.0)
- added Q4: BC547, myAmp:TO-92_Inline_Wide, F.Cu at (73.0, 115.9)
- added Q5: BC557, myAmp:TO-92_Inline_Wide, F.Cu at (44.4, 121.5)
- added R41: 4K7, myAmp:R_10MM, F.Cu at (35.8, 111.4)
- added R42: 4K7, myAmp:R_10MM, F.Cu at (48.6, 111.4)
- added R43: 10, myAmp:R_10MM, F.Cu at (61.4, 111.4)
- added R44: 10, myAmp:R_10MM, F.Cu at (74.1, 111.4)
- added R45: 20K, myAmp:R_10MM, F.Cu at (82.5, 87.0)
- added R46: 20K, myAmp:R_10MM, F.Cu at (82.5, 89.5)
- added SW5: disc/TLE2426, myAmp:ESP2010_switch, F.Cu at (35.0, 120.5)
- added U15: modulo-bus, myAmp:modulo-bus, F.Cu at (242.6, 3.17)
- added U16: modulo-bus, myAmp:modulo-bus, F.Cu at (47.2, 54.2)
- added U17: TLE2426, myAmp:TO-92_Inline_Wide, F.Cu at (52.0, 118.4)
- C11, C13, C14, C15, C17, C18, C19, C21, C23, C29, C30, C31, C34, C36, C49, C5, C50, C6, C9: footprint myAmp:C_1206 -> myAmp:C_5MM_1206
- C26, C27, C4: footprint myAmp:C_1206 -> myAmp:C_2.5MM
- D3, D6: footprint myAmp:LED_D3.0mm -> myAmp:LED_D3.0mm_PCBedge
- L1, L2, L3, L4: footprint myAmp:COILCRAFT_DR0810 -> myAmp:COILCRAFT_RFS1412
- RV4: renamed from RV6; footprint myAmp:ALPS_RK09L -> myAmp:BOURNS_PTD901_xx15K
- RV5: footprint myAmp:ALPS_RK09L -> myAmp:BOURNS_PTD901_xx15K
- RV6: renamed from RV4; footprint myAmp:ALPS_RK09L -> myAmp:BOURNS_PTD901_xx15K
- RV7: footprint myAmp:ALPS_RK09L_DBL -> myAmp:BOURNS_PTD902_xx15K
- RV8: value 10K -> 20K; footprint myAmp:ALPS_RK09L_DBL -> myAmp:BOURNS_PTD902_xx15K
- U6: value NE5532 -> modulo-bus; footprint myAmp:SOIC-8_3.9x4.9mm_P1.27mm -> myAmp:modulo-bus
- moved U6 103.1 mm to (139.7, 3.17)
- moved D3 63.5 mm to (234.3, 50.0)
- moved J4 60.5 mm to (194.3, 67.3), turned to 180 degrees
- moved C49 57.9 mm to (220.3, 19.1), turned to 90 degrees
- moved C50 57.2 mm to (224.8, 19.1), turned to 90 degrees
- moved L4 52.8 mm to (181.6, 42.5)
- moved RV8 51.1 mm to (82.5, 93.3)
- moved C36 50.5 mm to (120.7, 33.0), turned to 180 degrees
- moved C30 50.2 mm to (120.7, 26.7), turned to 180 degrees
- moved D6 50.2 mm to (116.2, 50.2)
- moved S2 47.7 mm to (196.8, 35.6), turned to 90 degrees
- moved R20 45.2 mm to (233.7, 31.8), turned to 180 degrees
- moved R40 44.3 mm to (233.7, 23.5), turned to 180 degrees
- moved C6 43.9 mm to (274.7, 11.8), turned to 90 degrees
- moved S1 42.8 mm to (196.8, 25.4), turned to 90 degrees
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Connections:
- net /pre amp/PREAMP_OUT renamed /pre amp/PA_OUT
- net LOUT renamed Net-(R45-Pad2)
- net Net-(C15-Pad1) renamed /FV-1/REFP
- net ROUT renamed Net-(R46-Pad2)
- C18 pad 1: /mixer/FV_LOUT -> /mixer/FVL
- C19 pad 1: /mixer/TONE_OUT -> /mixer/PAL
- C21 pad 1: /mixer/FV_ROUT -> /mixer/FVR
- C23 pad 1: /mixer/TONE_OUT -> /mixer/PAR
- C24 pad 2: VDD -> +12V
- C28 pad 1: VDD -> +12V
- C29 pad 1: VDD -> +12V
- C32 pad 1: VDD -> +12V
- C37 pad 1: VDD -> +12V
- C38 pad 1: VDD -> +12V
- C39 pad 1: VDD -> +12V
- C40 pad 1: VDD -> +12V
- D6 pad 2: VDD -> +12V
- R33 pad 1: VDD -> +12V
- R34 pad 1: VDD -> +12V
- SW2 pad 1: VDD -> +12V
- U12 pad 15: VDD -> +12V
- U12 pad 16: VDD -> +12V
- U12 pad 27: VDD -> +12V
- U12 pad 28: VDD -> +12V
- U12 pad 7: VDD -> +12V
- U13 pad 1: Net-(U13-Pad1) -> GND
- U13 pad 3: Net-(U13-Pad3) -> +12V
- U13 pad 5: Net-(U13-Pad5) -> +3V3
- U4 pad 3: VGND -> /mixer/MIX_VGND
- U4 pad 4: (no net) -> GND
- U4 pad 5: VGND -> /mixer/MIX_VGND
- U4 pad 8: (no net) -> +12V
- U6 pad 1: (no net) -> GND
- U6 pad 2: (no net) -> Net-(U6-Pad2)
- U6 pad 3: (no net) -> +12V
- U6 pad 4: GND -> Net-(U6-Pad4)
- U6 pad 5: (no net) -> Net-(U6-Pad5)
- U6 pad 6: (no net) -> Net-(U6-Pad6)
- U6 pad 7: (no net) -> Net-(U6-Pad7)
- U6 pad 8: VDD -> Net-(U6-Pad8)
- U7 pad 3: VDD -> +12V

Commit message: more layout
Parts:
- removed J16, J17, J18, J19: HOLE, myAmp:MountingHole
- added R47: 10K, myAmp:R_10MM, F.Cu at (261.6, 15.2)
- moved SW1 127.5 mm to (139.4, 104.1)
- moved C27 127.5 mm to (121.6, 124.4)
- moved C35 127.5 mm to (121.6, 121.5)
- moved R32 127.5 mm to (109.5, 115.2)
- moved RN3 127.5 mm to (126.9, 121.9)
- moved SS1 127.5 mm to (110.0, 104.6)
- moved C26 127.5 mm to (112.8, 118.0)
- moved J2 127.5 mm to (114.3, 121.8)
- moved SS2 127.5 mm to (123.8, 104.6)
- moved U9 127.5 mm to (106.8, 120.9)
- moved Y2 127.5 mm to (122.0, 116.9)
- moved RN1 127.5 mm to (148.9, 117.8)
- moved RN2 127.5 mm to (144.1, 114.8)
- moved RN4 127.5 mm to (144.1, 118.7)
- moved U10 127.5 mm to (152.8, 100.4)
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Connections:
- R45 pad 2: Net-(R45-Pad2) -> /mixer/MIXL
- R46 pad 2: Net-(R46-Pad2) -> /mixer/MIXR
- RV7 pad 2: VGND -> /mixer/MIX_VGND
- RV7 pad 5: VGND -> /mixer/MIX_VGND
- RV8 pad 2: Net-(R45-Pad2) -> /mixer/MIXL
- RV8 pad 3: Net-(R45-Pad2) -> /mixer/MIXL
- RV8 pad 5: Net-(R46-Pad2) -> /mixer/MIXR
- RV8 pad 6: Net-(R46-Pad2) -> /mixer/MIXR
- U16 pad 16: Net-(U16-Pad16) -> /mixer/MIXL
- U16 pad 17: Net-(U16-Pad17) -> GND
- U16 pad 18: Net-(U16-Pad18) -> /mixer/MIXR
- U16 pad 19: Net-(U16-Pad19) -> GND
- U4 pad 1: Net-(R45-Pad2) -> /mixer/MIXL
- U4 pad 7: Net-(R46-Pad2) -> /mixer/MIXR
- U5 pad 1: GND -> /FV-1/A0
Other:
- board size 302 x 101 mm -> 302 x 135 mm
- board text added: "FV-1 DSP"
- board text added: "mixer"
- board text added: "power amp"
- board text added: "power and AVR"
- board text added: "pre-amp"
