File: circuit/modulo.kicad_pcb (KiCad board)
At the start: 4 copper layers, 302 x 135 mm, 184 parts, among them J1 JACK_MONO, J10 HOLE, J11 HOLE, J12 HOLE, J13 HOLE, J14 HOLE, J15 HOLE, J2 CONN_01X03, J20 HOLE, J21 HOLE, J22 HOLE, J23 HOLE, J24 HOLE, J25 HOLE, J26 HOLE, J27 HOLE, J3 HOLE, J4 Barrel_Jack_Switch, J5 HOLE, J6 HOLE, J7 HOLE, J8 HOLE, J9 HOLE, Q1 MMBFJ201, Q2 BC547, Q3 BC557, Q4 BC547, Q5 BC557, SW1 ROT_SW, SW2 ON/OFF, SW3 Idss/Vp, SW4 disc/TLE2426, SW5 disc/TLE2426, U1 TLE2426, U10 74164, U11 74164, U12 TPA3136D2, U13 modulo-bus, U14 modulo-bus, U15 modulo-bus, U16 modulo-bus, U17 TLE2426, U2 NE5532, U3 FV-1, U4 NE5532, U5 24LC32A, U6 modulo-bus, U7 LM1117, U8 ATMEGA8, U9 AVR-ISP6, Y1 32768Hz, Y2 8MHz

Commit message: even more layout
Parts:
- removed J20, J21, J22, J23: HOLE, myAmp:MountingHole
- removed RN4: 100, myAmp:R_Array_x4_1206
- removed SS1, SS2: SEVSEG, myAmp:7seg_14.2mm
- added D10: 1, myAmp:LED_D3.0mm_PCBedge, F.Cu at (111.1, 134.6)
- added D11: 2, myAmp:LED_D3.0mm_PCBedge, F.Cu at (116.2, 134.6)
- added D12: 3, myAmp:LED_D3.0mm_PCBedge, F.Cu at (121.3, 134.6)
- added D13: 4, myAmp:LED_D3.0mm_PCBedge, F.Cu at (126.4, 134.6)
- added D14: 5, myAmp:LED_D3.0mm_PCBedge, F.Cu at (131.4, 134.6)
- added D15: 6, myAmp:LED_D3.0mm_PCBedge, F.Cu at (136.5, 134.6)
- added D16: 7, myAmp:LED_D3.0mm_PCBedge, F.Cu at (141.6, 134.6)
- added D17: 8, myAmp:LED_D3.0mm_PCBedge, F.Cu at (146.7, 134.6)
- added D18: 9, myAmp:LED_D3.0mm_PCBedge, F.Cu at (156.2, 134.6)
- added D19: 10, myAmp:LED_D3.0mm_PCBedge, F.Cu at (161.3, 134.6)
- added D20: 11, myAmp:LED_D3.0mm_PCBedge, F.Cu at (166.4, 134.6)
- added D21: 12, myAmp:LED_D3.0mm_PCBedge, F.Cu at (171.4, 134.6)
- added J17: HOLE, myAmp:MountingHole, F.Cu at (197.0, 131.0)
- added J18: HOLE, myAmp:MountingHole, F.Cu at (197.0, 89.0)
- added J19: HOLE, myAmp:MountingHole, F.Cu at (105.0, 89.0)
- added U18: DBG_UART, myAmp:DBG_UART, F.Cu at (156.2, 91.4)
- J2: value CONN_01X03 -> Barrel_Jack_Switch; footprint myAmp:PIN_1x03 -> myAmp:POWER_JACK_2.1mm
- J4: value Barrel_Jack_Switch -> HOLE; footprint myAmp:POWER_JACK_2.1mm -> myAmp:MountingHole
- RN1, RN2, RN3: footprint myAmp:R_Array_x4_1206 -> myAmp:R_Array_x4_P2.54
- SW1: value ROT_SW -> ON/OFF; footprint myAmp:ROT_ENC -> myAmp:ESP2010_switch
- SW2: value ON/OFF -> ROT_SW; footprint myAmp:ESP2010_switch -> myAmp:BOURNS_PEC12R_2x17F
- U10: value 74164 -> AVR-ISP6; footprint myAmp:SOIC-14_3.9x8.7mm_P1.27mm -> myAmp:AVR_ISP6
- U13: value modulo-bus -> 74164; footprint myAmp:modulo-bus -> myAmp:SOIC-14_3.9x8.7mm_P1.27mm
- U8: value ATMEGA8 -> modulo-bus; footprint myAmp:TQFP-32_7x7mm_Pitch0.8mm -> myAmp:modulo-bus
- U9: value AVR-ISP6 -> ATMEGA8; footprint myAmp:AVR_ISP6 -> myAmp:TQFP-32_7x7mm_Pitch0.8mm
- moved J4 87.2 mm to (105.0, 131.0), turned to 0 degrees
- moved J2 68.8 mm to (181.0, 104.8)
- moved C35 66.1 mm to (180.1, 90.6)
- moved R33 60.2 mm to (115.1, 101.8)
- moved U9 57.4 mm to (159.6, 98.6)
- moved U13 39.2 mm to (160.7, 121.3), turned to 90 degrees
- moved C27 39.2 mm to (151.3, 98.9)
- moved RN3 37.4 mm to (163.8, 127.6)
- moved R32 36.9 mm to (142.7, 99.1)
- moved RN1 31.7 mm to (118.7, 127.6)
- moved U8 30.9 mm to (139.0, 87.6)
- moved U7 27.7 mm to (141.3, 104.3)
- moved SW1 26.5 mm to (114.3, 112.5)
- moved C26 26.5 mm to (138.9, 113.1)
- moved U11 24.8 mm to (130.0, 120.7)
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Connections:
- C25 pad 1: +3V3 -> Net-(C25-Pad1)
- J2 pad 1: GND -> Net-(J2-Pad1)
- J2 pad 2: +3V3 -> GND
- J2 pad 3: /mcu/DBG_TX -> GND
- R32 pad 1: /mcu/AVR_RST -> /power and MCU/AVR_RST
- RN1 pad 2: Net-(RN1-Pad2) -> Net-(D10-Pad2)
- RN1 pad 4: Net-(RN1-Pad4) -> Net-(D11-Pad2)
- RN2 pad 2: Net-(RN2-Pad2) -> Net-(D14-Pad2)
- RN2 pad 4: Net-(RN2-Pad4) -> Net-(D15-Pad2)
- RN3 pad 2: Net-(RN3-Pad2) -> Net-(D18-Pad2)
- RN3 pad 4: Net-(RN3-Pad4) -> Net-(D19-Pad2)
- SW1 pad 1: Net-(SW1-Pad1) -> +12V
- SW1 pad 2: GND -> Net-(J2-Pad1)
- SW1 pad 3: Net-(SW1-Pad3) -> (no net)
- SW2 pad 1: +12V -> Net-(SW2-Pad1)
- SW2 pad 2: Net-(J4-Pad1) -> GND
- SW2 pad 3: (no net) -> Net-(SW2-Pad3)
- U10 pad 1: /mcu/LED_DT -> /power and MCU/MISO
- U10 pad 2: /mcu/LED_DT -> +3V3
- U10 pad 3: Net-(RN1-Pad1) -> /power and MCU/SCK
- U10 pad 4: Net-(RN1-Pad2) -> /power and MCU/MOSI
- U10 pad 5: Net-(RN1-Pad3) -> /power and MCU/AVR_RST
- U10 pad 6: Net-(RN1-Pad4) -> GND
- U11 pad 1: Net-(RN2-Pad1) -> /power and MCU/LED_DT
- U11 pad 10: Net-(RN4-Pad4) -> Net-(RN2-Pad1)
- U11 pad 11: Net-(RN4-Pad3) -> Net-(RN2-Pad3)
- U11 pad 12: Net-(RN4-Pad2) -> Net-(RN2-Pad5)
- U11 pad 13: Net-(RN4-Pad1) -> Net-(RN2-Pad7)
- U11 pad 2: Net-(RN2-Pad1) -> /power and MCU/LED_DT
- U11 pad 3: Net-(RN3-Pad1) -> Net-(RN1-Pad1)
- U11 pad 4: Net-(RN3-Pad2) -> Net-(RN1-Pad3)
- U11 pad 5: Net-(RN3-Pad3) -> Net-(RN1-Pad5)
- U11 pad 6: Net-(RN3-Pad4) -> Net-(RN1-Pad7)
- U11 pad 8: /mcu/LED_CK -> /power and MCU/LED_CK
- U11 pad 9: /mcu/LED_RST -> /power and MCU/LED_RST
- U13 pad 1: GND -> Net-(RN2-Pad7)
- U13 pad 14: Net-(U13-Pad14) -> +3V3
- U13 pad 2: Net-(U13-Pad2) -> Net-(RN2-Pad7)
- U13 pad 3: +12V -> Net-(RN3-Pad1)
- U13 pad 4: Net-(U13-Pad4) -> Net-(RN3-Pad3)
- U13 pad 5: +3V3 -> Net-(RN3-Pad5)
- U13 pad 6: Net-(U13-Pad6) -> Net-(RN3-Pad7)
- U13 pad 7: Net-(U13-Pad7) -> GND
- U13 pad 8: Net-(U13-Pad8) -> /power and MCU/LED_CK
- U13 pad 9: Net-(U13-Pad9) -> /power and MCU/LED_RST
- U8 pad 1: /mcu/LED_CK -> GND
- U8 pad 10: Net-(SW1-Pad1) -> Net-(U8-Pad10)
- U8 pad 11: /mcu/ROT_SW -> Net-(U8-Pad11)
- U8 pad 15: /mcu/MOSI -> Net-(U8-Pad15)
- U8 pad 16: /mcu/MISO -> Net-(U8-Pad16)
- U8 pad 17: /mcu/SCK -> Net-(U8-Pad17)
- U8 pad 18: +3V3 -> Net-(U8-Pad18)
- U8 pad 2: /mcu/LED_RST -> Net-(U8-Pad2)
- U8 pad 20: +3V3 -> Net-(U8-Pad20)
- U8 pad 3: GND -> +12V
- U8 pad 4: +3V3 -> Net-(U8-Pad4)
- U8 pad 5: GND -> +3V3
- U8 pad 6: +3V3 -> Net-(U8-Pad6)
- U8 pad 7: Net-(C26-Pad1) -> Net-(U8-Pad7)
- U8 pad 8: Net-(C27-Pad1) -> Net-(U8-Pad8)
- U8 pad 9: Net-(SW1-Pad3) -> Net-(U8-Pad9)
- U9 pad 1: /mcu/MISO -> /power and MCU/LED_CK
- U9 pad 2: +3V3 -> /power and MCU/LED_RST
- U9 pad 3: /mcu/SCK -> GND
- U9 pad 4: /mcu/MOSI -> +3V3
- U9 pad 5: /mcu/AVR_RST -> GND
- U9 pad 6: GND -> +3V3
Other:
- board text added: "fv-1 dsp"
- board text added: "power and mcu"
- board text removed: "FV-1 DSP"
- board text removed: "power and AVR"

Commit message: small updates
Parts:
- moved SW1 85.2 mm to (199.4, 109.9), turned to 270 degrees
- moved R33 56.8 mm to (171.4, 94.6)
- moved U10 49.7 mm to (196.8, 120.0)
- moved Y2 47.6 mm to (172.7, 116.8), turned to 270 degrees
- moved R32 35.2 mm to (176.5, 108.6), turned to 180 degrees
- moved C26 29.4 mm to (168.3, 114.3), turned to 270 degrees
- moved U9 27.9 mm to (182.2, 114.9)
- moved U18 26.6 mm to (178.4, 106.0)
- moved C27 26.1 mm to (168.3, 118.7), turned to 90 degrees
- moved C35 25.1 mm to (189.9, 113.7), turned to 270 degrees
- moved C25 18.5 mm to (134.0, 99.7), turned to 180 degrees
- moved J2 13.1 mm to (192.4, 98.4), turned to 180 degrees
- moved U7 7.65 mm to (134.0, 106.7)
- moved U13 3.81 mm to (156.8, 121.3)
Connections:
- C25 pad 1: Net-(C25-Pad1) -> +3V3
- J10 pad 1: Net-(J10-Pad1) -> (no net)
- J11 pad 1: Net-(J11-Pad1) -> (no net)
- J12 pad 1: Net-(J12-Pad1) -> (no net)
- J13 pad 1: Net-(J13-Pad1) -> (no net)
- J14 pad 1: Net-(J14-Pad1) -> (no net)
- J15 pad 1: Net-(J15-Pad1) -> (no net)
- J17 pad 1: Net-(J17-Pad1) -> (no net)
- J18 pad 1: Net-(J18-Pad1) -> (no net)
- J19 pad 1: Net-(J19-Pad1) -> (no net)
- J24 pad 1: Net-(J24-Pad1) -> (no net)
- J25 pad 1: Net-(J25-Pad1) -> (no net)
- J26 pad 1: Net-(J26-Pad1) -> (no net)
- J27 pad 1: Net-(J27-Pad1) -> (no net)
- J3 pad 1: Net-(J3-Pad1) -> (no net)
- J4 pad 1: Net-(J4-Pad1) -> (no net)
- J5 pad 1: Net-(J5-Pad1) -> (no net)
- J6 pad 1: Net-(J6-Pad1) -> (no net)
- J7 pad 1: Net-(J7-Pad1) -> (no net)
- J8 pad 1: Net-(J8-Pad1) -> (no net)
- J9 pad 1: Net-(J9-Pad1) -> (no net)
- U12 pad 13: Net-(U12-Pad13) -> (no net)
- U12 pad 5: Net-(U12-Pad5) -> (no net)
- U12 pad 6: Net-(U12-Pad6) -> (no net)
- U13 pad 10: Net-(U13-Pad10) -> (no net)
- U13 pad 11: Net-(U13-Pad11) -> (no net)
- U13 pad 12: Net-(U13-Pad12) -> (no net)
- U13 pad 13: Net-(U13-Pad13) -> (no net)
- U14 pad 10: Net-(U14-Pad10) -> (no net)
- U14 pad 11: Net-(U14-Pad11) -> (no net)
- U14 pad 12: Net-(U14-Pad12) -> (no net)
- U14 pad 13: Net-(U14-Pad13) -> (no net)
- U14 pad 14: Net-(U14-Pad14) -> (no net)
- U14 pad 15: Net-(U14-Pad15) -> (no net)
- U14 pad 16: Net-(U14-Pad16) -> (no net)
- U14 pad 17: Net-(U14-Pad17) -> (no net)
- U14 pad 18: Net-(U14-Pad18) -> (no net)
- U14 pad 19: Net-(U14-Pad19) -> (no net)
- U14 pad 2: Net-(U14-Pad2) -> (no net)
- U14 pad 20: Net-(U14-Pad20) -> (no net)
- U14 pad 4: Net-(U14-Pad4) -> (no net)
- U14 pad 5: Net-(U14-Pad5) -> (no net)
- U14 pad 8: Net-(U14-Pad8) -> (no net)
- U14 pad 9: Net-(U14-Pad9) -> (no net)
- U15 pad 16: Net-(U15-Pad16) -> (no net)
- U15 pad 17: Net-(U15-Pad17) -> (no net)
- U15 pad 18: Net-(U15-Pad18) -> (no net)
- U15 pad 19: Net-(U15-Pad19) -> (no net)
- U15 pad 2: Net-(U15-Pad2) -> (no net)
- U15 pad 3: Net-(U15-Pad3) -> (no net)
- U15 pad 4: Net-(U15-Pad4) -> (no net)
- U16 pad 10: Net-(U16-Pad10) -> (no net)
- U16 pad 11: Net-(U16-Pad11) -> (no net)
- U16 pad 12: Net-(U16-Pad12) -> (no net)
- U16 pad 13: Net-(U16-Pad13) -> (no net)
- U16 pad 14: Net-(U16-Pad14) -> (no net)
- U16 pad 15: Net-(U16-Pad15) -> (no net)
- U16 pad 2: Net-(U16-Pad2) -> (no net)
- U16 pad 20: Net-(U16-Pad20) -> (no net)
- U16 pad 4: Net-(U16-Pad4) -> (no net)
- U16 pad 5: Net-(U16-Pad5) -> (no net)
- U6 pad 10: Net-(U6-Pad10) -> (no net)
- U6 pad 11: Net-(U6-Pad11) -> (no net)
- U6 pad 12: Net-(U6-Pad12) -> (no net)
- U6 pad 13: Net-(U6-Pad13) -> (no net)
- U6 pad 14: Net-(U6-Pad14) -> (no net)
- U6 pad 15: Net-(U6-Pad15) -> (no net)
- U6 pad 2: Net-(U6-Pad2) -> (no net)
- U6 pad 20: Net-(U6-Pad20) -> (no net)
- U6 pad 4: Net-(U6-Pad4) -> (no net)
- U6 pad 5: Net-(U6-Pad5) -> (no net)
- U6 pad 6: Net-(U6-Pad6) -> (no net)
- U6 pad 7: Net-(U6-Pad7) -> (no net)
- U6 pad 8: Net-(U6-Pad8) -> (no net)
- U6 pad 9: Net-(U6-Pad9) -> (no net)
- U8 pad 10: Net-(U8-Pad10) -> (no net)
- U8 pad 11: Net-(U8-Pad11) -> (no net)
- U8 pad 12: Net-(U8-Pad12) -> (no net)
- U8 pad 13: Net-(U8-Pad13) -> (no net)
- U8 pad 14: Net-(U8-Pad14) -> (no net)
- U8 pad 15: Net-(U8-Pad15) -> (no net)
- U8 pad 16: Net-(U8-Pad16) -> (no net)
- U8 pad 17: Net-(U8-Pad17) -> (no net)
- U8 pad 18: Net-(U8-Pad18) -> (no net)
- U8 pad 19: Net-(U8-Pad19) -> (no net)
- U8 pad 2: Net-(U8-Pad2) -> (no net)
- U8 pad 20: Net-(U8-Pad20) -> (no net)
- U8 pad 4: Net-(U8-Pad4) -> (no net)
- U8 pad 6: Net-(U8-Pad6) -> (no net)
- U8 pad 7: Net-(U8-Pad7) -> (no net)
- U8 pad 8: Net-(U8-Pad8) -> (no net)
- U8 pad 9: Net-(U8-Pad9) -> (no net)
- U9 pad 12: Net-(U9-Pad12) -> (no net)
- U9 pad 13: Net-(U9-Pad13) -> (no net)
- U9 pad 14: Net-(U9-Pad14) -> (no net)
- U9 pad 19: Net-(U9-Pad19) -> (no net)
- U9 pad 22: Net-(U9-Pad22) -> (no net)
- U9 pad 23: /power and MCU/S2 -> (no net)
- U9 pad 24: /power and MCU/S1 -> (no net)
- U9 pad 25: /power and MCU/S0 -> (no net)
- U9 pad 26: /power and MCU/T0 -> (no net)
- U9 pad 27: /power and MCU/SDA -> (no net)
- U9 pad 28: /power and MCU/SCL -> (no net)
- U9 pad 30: /power and MCU/WP -> (no net)

Commit message: added DC-DC converter
Parts:
- added C55: 4.7µf, myAmp:CPOL_D4_P1.5, F.Cu at (116.2, 105.4)
- added C56: 100nF, myAmp:C_5MM_1206, F.Cu at (121.9, 104.1)
- added C57: 100nF, myAmp:C_1206, F.Cu at (116.2, 97.2)
- added C58: 15µf, myAmp:C_1812, F.Cu at (130.8, 103.5)
- added C59: 15µf, myAmp:C_1812, F.Cu at (127.0, 103.5)
- added L5: 68µH, myAmp:COIL_SRR6603, F.Cu at (124.5, 97.2)
- added R48: 75K, myAmp:R_10MM, F.Cu at (117.5, 94.0)
- added R49: 10K, myAmp:R_10MM, F.Cu at (112.4, 105.4)
- added R50: 10K, myAmp:R_10MM, F.Cu at (109.9, 105.4)
- added U19: TPS560430, myAmp:SOT-23-6, F.Cu at (116.2, 101.3)
- moved U7 11.8 mm to (135.3, 94.9)
- moved C25 1.80 mm to (135.3, 101.0)
Connections:
- J10 pad 1: (no net) -> Net-(J10-Pad1)
- J11 pad 1: (no net) -> Net-(J11-Pad1)
- J12 pad 1: (no net) -> Net-(J12-Pad1)
- J13 pad 1: (no net) -> Net-(J13-Pad1)
- J14 pad 1: (no net) -> Net-(J14-Pad1)
- J15 pad 1: (no net) -> Net-(J15-Pad1)
- J17 pad 1: (no net) -> Net-(J17-Pad1)
- J18 pad 1: (no net) -> Net-(J18-Pad1)
- J19 pad 1: (no net) -> Net-(J19-Pad1)
- J24 pad 1: (no net) -> Net-(J24-Pad1)
- J25 pad 1: (no net) -> Net-(J25-Pad1)
- J26 pad 1: (no net) -> Net-(J26-Pad1)
- J27 pad 1: (no net) -> Net-(J27-Pad1)
- J3 pad 1: (no net) -> Net-(J3-Pad1)
- J4 pad 1: (no net) -> Net-(J4-Pad1)
- J5 pad 1: (no net) -> Net-(J5-Pad1)
- J6 pad 1: (no net) -> Net-(J6-Pad1)
- J7 pad 1: (no net) -> Net-(J7-Pad1)
- J8 pad 1: (no net) -> Net-(J8-Pad1)
- J9 pad 1: (no net) -> Net-(J9-Pad1)
- U12 pad 13: (no net) -> Net-(U12-Pad13)
- U12 pad 5: (no net) -> Net-(U12-Pad5)
- U12 pad 6: (no net) -> Net-(U12-Pad6)
- U13 pad 10: (no net) -> Net-(U13-Pad10)
- U13 pad 11: (no net) -> Net-(U13-Pad11)
- U13 pad 12: (no net) -> Net-(U13-Pad12)
- U13 pad 13: (no net) -> Net-(U13-Pad13)
- U14 pad 10: (no net) -> Net-(U14-Pad10)
- U14 pad 11: (no net) -> Net-(U14-Pad11)
- U14 pad 12: (no net) -> Net-(U14-Pad12)
- U14 pad 13: (no net) -> Net-(U14-Pad13)
- U14 pad 14: (no net) -> Net-(U14-Pad14)
- U14 pad 15: (no net) -> Net-(U14-Pad15)
- U14 pad 16: (no net) -> Net-(U14-Pad16)
- U14 pad 17: (no net) -> Net-(U14-Pad17)
- U14 pad 18: (no net) -> Net-(U14-Pad18)
- U14 pad 19: (no net) -> Net-(U14-Pad19)
- U14 pad 2: (no net) -> Net-(U14-Pad2)
- U14 pad 20: (no net) -> Net-(U14-Pad20)
- U14 pad 4: (no net) -> Net-(U14-Pad4)
- U14 pad 5: (no net) -> Net-(U14-Pad5)
- U14 pad 8: (no net) -> Net-(U14-Pad8)
- U14 pad 9: (no net) -> Net-(U14-Pad9)
- U15 pad 16: (no net) -> Net-(U15-Pad16)
- U15 pad 17: (no net) -> Net-(U15-Pad17)
- U15 pad 18: (no net) -> Net-(U15-Pad18)
- U15 pad 19: (no net) -> Net-(U15-Pad19)
- U15 pad 2: (no net) -> Net-(U15-Pad2)
- U15 pad 3: (no net) -> Net-(U15-Pad3)
- U15 pad 4: (no net) -> Net-(U15-Pad4)
- U16 pad 10: (no net) -> Net-(U16-Pad10)
- U16 pad 11: (no net) -> Net-(U16-Pad11)
- U16 pad 12: (no net) -> Net-(U16-Pad12)
- U16 pad 13: (no net) -> Net-(U16-Pad13)
- U16 pad 14: (no net) -> Net-(U16-Pad14)
- U16 pad 15: (no net) -> Net-(U16-Pad15)
- U16 pad 2: (no net) -> Net-(U16-Pad2)
- U16 pad 20: (no net) -> Net-(U16-Pad20)
- U16 pad 4: (no net) -> Net-(U16-Pad4)
- U16 pad 5: (no net) -> Net-(U16-Pad5)
- U6 pad 10: (no net) -> Net-(U6-Pad10)
- U6 pad 11: (no net) -> Net-(U6-Pad11)
- U6 pad 12: (no net) -> Net-(U6-Pad12)
- U6 pad 13: (no net) -> Net-(U6-Pad13)
- U6 pad 14: (no net) -> Net-(U6-Pad14)
- U6 pad 15: (no net) -> Net-(U6-Pad15)
- U6 pad 2: (no net) -> Net-(U6-Pad2)
- U6 pad 20: (no net) -> Net-(U6-Pad20)
- U6 pad 4: (no net) -> Net-(U6-Pad4)
- U6 pad 5: (no net) -> Net-(U6-Pad5)
- U6 pad 6: (no net) -> Net-(U6-Pad6)
- U6 pad 7: (no net) -> Net-(U6-Pad7)
- U6 pad 8: (no net) -> Net-(U6-Pad8)
- U6 pad 9: (no net) -> Net-(U6-Pad9)
- U7 pad 3: +12V -> /power and MCU/4.75V
- U8 pad 10: (no net) -> Net-(U8-Pad10)
- U8 pad 11: (no net) -> Net-(U8-Pad11)
- U8 pad 12: (no net) -> Net-(U8-Pad12)
- U8 pad 13: (no net) -> Net-(U8-Pad13)
- U8 pad 14: (no net) -> Net-(U8-Pad14)
- U8 pad 15: (no net) -> Net-(U8-Pad15)
- U8 pad 16: (no net) -> Net-(U8-Pad16)
- U8 pad 17: (no net) -> Net-(U8-Pad17)
- U8 pad 18: (no net) -> Net-(U8-Pad18)
- U8 pad 19: (no net) -> Net-(U8-Pad19)
- U8 pad 2: (no net) -> Net-(U8-Pad2)
- U8 pad 20: (no net) -> Net-(U8-Pad20)
- U8 pad 4: (no net) -> Net-(U8-Pad4)
- U8 pad 6: (no net) -> Net-(U8-Pad6)
- U8 pad 7: (no net) -> Net-(U8-Pad7)
- U8 pad 8: (no net) -> Net-(U8-Pad8)
- U8 pad 9: (no net) -> Net-(U8-Pad9)
- U9 pad 12: (no net) -> Net-(U9-Pad12)
- U9 pad 13: (no net) -> Net-(U9-Pad13)
- U9 pad 14: (no net) -> Net-(U9-Pad14)
- U9 pad 19: (no net) -> Net-(U9-Pad19)
- U9 pad 22: (no net) -> Net-(U9-Pad22)
- U9 pad 23: (no net) -> /power and MCU/S2
- U9 pad 24: (no net) -> /power and MCU/S1
- U9 pad 25: (no net) -> /power and MCU/S0
- U9 pad 26: (no net) -> /power and MCU/T0
- U9 pad 27: (no net) -> /power and MCU/SDA
- U9 pad 28: (no net) -> /power and MCU/SCL
- U9 pad 30: (no net) -> /power and MCU/WP
