File: circuit/modulo.kicad_pcb (KiCad board)
At the start: 2 copper layers, 302 x 135 mm, 201 parts, among them J1 JACK_MONO, J10 HOLE, J11 HOLE, J12 HOLE, J13 HOLE, J14 HOLE, J15 HOLE, J17 HOLE, J18 HOLE, J19 HOLE, J2 Barrel_Jack_Switch, J24 HOLE, J25 HOLE, J26 HOLE, J27 HOLE, J3 HOLE, J4 HOLE, J5 HOLE, J6 HOLE, J7 HOLE, J8 HOLE, J9 HOLE, Q1 MMBFJ201, Q2 BC547, Q3 BC557, Q4 BC547, Q5 BC557, SW1 OFF/ON, SW2 ROT_SW, SW3 Idss/Vp, SW4 disc/TLE2426, SW5 disc/TLE2426, U1 TLE2426, U10 AVR-ISP6, U11 74164, U12 TPA3136D2, U13 74164, U14 modulo-bus, U15 modulo-bus, U16 modulo-bus, U17 TLE2426, U18 DBG_UART, U19 TPS560430, U2 NE5532, U3 FV-1, U4 NE5532, U5 24LC32A, U6 modulo-bus, U7 LM1117, U8 modulo-bus, U9 ATMEGA8, Y1 32768Hz, Y2 8MHz

Commit message: routed FV-1 and the mixer
Parts:
- moved SW5 83.8 mm to (3.17, 97.8), turned to 90 degrees
- moved C52 69.4 mm to (19.7, 109.9)
- moved C53 69.4 mm to (12.1, 109.9)
- moved D9 69.4 mm to (12.1, 121.3)
- moved R41 69.4 mm to (22.2, 121.3)
- moved R43 69.4 mm to (17.1, 121.3)
- moved U17 69.4 mm to (15.9, 102.2)
- moved R42 69.4 mm to (9.53, 121.3)
- moved R44 69.4 mm to (14.6, 121.3)
- moved D8 69.4 mm to (19.7, 121.3)
- moved Q4 69.4 mm to (19.7, 130.2)
- moved Q5 69.4 mm to (12.1, 130.2)
- moved C54 59.7 mm to (17.8, 96.5), turned to 0 degrees
- moved D3 52.5 mm to (286.8, 50.0)
- moved R3 38.4 mm to (274.3, 29.8), turned to 180 degrees
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Connections:
- C3 pad 2: /pre amp/vgnd_tle -> +12V
- C54 pad 2: /mixer/vgnd_tle -> +12V
- D18 pad 1: Net-(D18-Pad1) -> GND
- D19 pad 1: Net-(D18-Pad1) -> GND
- D20 pad 1: Net-(D18-Pad1) -> GND
- D21 pad 1: Net-(D18-Pad1) -> GND
- J10 pad 1: (no net) -> Net-(J10-Pad1)
- J11 pad 1: (no net) -> Net-(J11-Pad1)
- J12 pad 1: (no net) -> Net-(J12-Pad1)
- J13 pad 1: (no net) -> Net-(J13-Pad1)
- J14 pad 1: (no net) -> Net-(J14-Pad1)
- J15 pad 1: (no net) -> Net-(J15-Pad1)
- J17 pad 1: (no net) -> Net-(J17-Pad1)
- J18 pad 1: (no net) -> Net-(J18-Pad1)
- J19 pad 1: (no net) -> Net-(J19-Pad1)
- J24 pad 1: (no net) -> Net-(J24-Pad1)
- J25 pad 1: (no net) -> Net-(J25-Pad1)
- J26 pad 1: (no net) -> Net-(J26-Pad1)
- J27 pad 1: (no net) -> Net-(J27-Pad1)
- J3 pad 1: (no net) -> Net-(J3-Pad1)
- J4 pad 1: (no net) -> Net-(J4-Pad1)
- J5 pad 1: (no net) -> Net-(J5-Pad1)
- J6 pad 1: (no net) -> Net-(J6-Pad1)
- J7 pad 1: (no net) -> Net-(J7-Pad1)
- J8 pad 1: (no net) -> Net-(J8-Pad1)
- J9 pad 1: (no net) -> Net-(J9-Pad1)
- RV4 pad 1: +3V3 -> GND
- RV4 pad 3: GND -> +3V3
- RV5 pad 1: +3V3 -> GND
- RV5 pad 3: GND -> +3V3
- RV6 pad 1: +3V3 -> GND
- RV6 pad 3: GND -> +3V3
- U12 pad 13: (no net) -> Net-(U12-Pad13)
- U12 pad 5: (no net) -> Net-(U12-Pad5)
- U12 pad 6: (no net) -> Net-(U12-Pad6)
- U13 pad 10: (no net) -> Net-(U13-Pad10)
- U13 pad 11: (no net) -> Net-(U13-Pad11)
- U13 pad 12: (no net) -> Net-(U13-Pad12)
- U13 pad 13: (no net) -> Net-(U13-Pad13)
- U14 pad 10: (no net) -> Net-(U14-Pad10)
- U14 pad 11: (no net) -> Net-(U14-Pad11)
- U14 pad 12: (no net) -> Net-(U14-Pad12)
- U14 pad 13: (no net) -> Net-(U14-Pad13)
- U14 pad 14: (no net) -> Net-(U14-Pad14)
- U14 pad 15: (no net) -> Net-(U14-Pad15)
- U14 pad 16: (no net) -> Net-(U14-Pad16)
- U14 pad 17: (no net) -> Net-(U14-Pad17)
- U14 pad 18: (no net) -> Net-(U14-Pad18)
- U14 pad 19: (no net) -> Net-(U14-Pad19)
- U14 pad 2: (no net) -> Net-(U14-Pad2)
- U14 pad 20: (no net) -> Net-(U14-Pad20)
- U14 pad 21: (no net) -> Net-(U14-Pad21)
- U14 pad 4: (no net) -> Net-(U14-Pad4)
- U14 pad 5: (no net) -> Net-(U14-Pad5)
- U14 pad 8: (no net) -> Net-(U14-Pad8)
- U14 pad 9: (no net) -> Net-(U14-Pad9)
- U15 pad 16: (no net) -> Net-(U15-Pad16)
- U15 pad 17: (no net) -> Net-(U15-Pad17)
- U15 pad 18: (no net) -> Net-(U15-Pad18)
- U15 pad 19: (no net) -> Net-(U15-Pad19)
- U15 pad 2: (no net) -> Net-(U15-Pad2)
- U15 pad 3: (no net) -> Net-(U15-Pad3)
- U15 pad 4: (no net) -> Net-(U15-Pad4)
- U16 pad 10: (no net) -> Net-(U16-Pad10)
- U16 pad 11: (no net) -> Net-(U16-Pad11)
- U16 pad 12: (no net) -> Net-(U16-Pad12)
- U16 pad 13: (no net) -> Net-(U16-Pad13)
- U16 pad 14: (no net) -> Net-(U16-Pad14)
- U16 pad 15: (no net) -> Net-(U16-Pad15)
- U16 pad 2: (no net) -> Net-(U16-Pad2)
- U16 pad 20: (no net) -> Net-(U16-Pad20)
- U16 pad 21: (no net) -> Net-(U16-Pad21)
- U16 pad 4: (no net) -> Net-(U16-Pad4)
- U16 pad 5: (no net) -> Net-(U16-Pad5)
- U6 pad 10: (no net) -> Net-(U6-Pad10)
- U6 pad 11: (no net) -> Net-(U6-Pad11)
- U6 pad 12: (no net) -> Net-(U6-Pad12)
- U6 pad 13: (no net) -> Net-(U6-Pad13)
- U6 pad 14: (no net) -> Net-(U6-Pad14)
- U6 pad 15: (no net) -> Net-(U6-Pad15)
- U6 pad 2: (no net) -> Net-(U6-Pad2)
- U6 pad 20: (no net) -> Net-(U6-Pad20)
- U6 pad 21: (no net) -> Net-(U6-Pad21)
- U6 pad 4: (no net) -> Net-(U6-Pad4)
- U6 pad 5: (no net) -> Net-(U6-Pad5)
- U6 pad 6: (no net) -> Net-(U6-Pad6)
- U6 pad 7: (no net) -> Net-(U6-Pad7)
- U6 pad 8: (no net) -> Net-(U6-Pad8)
- U6 pad 9: (no net) -> Net-(U6-Pad9)
- U8 pad 16: (no net) -> Net-(U8-Pad16)
- U8 pad 17: (no net) -> Net-(U8-Pad17)
- U8 pad 18: (no net) -> Net-(U8-Pad18)
- U8 pad 19: (no net) -> Net-(U8-Pad19)
- U8 pad 2: (no net) -> Net-(U8-Pad2)
- U8 pad 4: (no net) -> Net-(U8-Pad4)
- U8 pad 6: (no net) -> Net-(U8-Pad6)
- U8 pad 7: (no net) -> Net-(U8-Pad7)
- U8 pad 8: (no net) -> Net-(U8-Pad8)
- U8 pad 9: (no net) -> Net-(U8-Pad9)
- U9 pad 1: (no net) -> Net-(U9-Pad1)
- U9 pad 2: (no net) -> Net-(U9-Pad2)
- U9 pad 30: (no net) -> Net-(U9-Pad30)
- U9 pad 32: (no net) -> Net-(U9-Pad32)
Routing:
- net +3V3: track 131.9 -> 334.3 mm
- net /mixer/MIXR: track 0.00 -> 80.9 mm
- net +12V: track 305.8 -> 384.1 mm
- net /mixer/MIX_VGND: track 0.00 -> 72.3 mm
- net /mixer/MIXL: track 0.00 -> 64.4 mm, vias 0 -> 1
- net Net-(R28-Pad2): track 0.00 -> 61.8 mm
- net Net-(RV6-Pad2): track 0.00 -> 55.2 mm
- net Net-(RV4-Pad2): track 0.00 -> 48.5 mm, vias 0 -> 1
- net Net-(R30-Pad2): track 0.00 -> 41.3 mm
- net /FV-1/FV_LIN: track 0.00 -> 39.1 mm
- net /mixer/vgnd_disc: track 0.00 -> 34.2 mm
- net /FV-1/FV_RIN: track 0.00 -> 33.8 mm
- net /FV-1/WP: track 0.00 -> 33.7 mm
- net /FV-1/S2: track 0.00 -> 32.5 mm
- net /FV-1/T0: track 0.00 -> 29.9 mm
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
Commit message: first routing done
Parts:
- moved C3 4.07 mm to (78.7, 14.6)
- moved R10 2.54 mm to (54.6, 14.0)
- moved R11 2.54 mm to (57.1, 14.0)
- turned C2 to 180 degrees
Routing:
- net +12V: track 384.1 -> 508.1 mm
- net /pre amp/PA_VGND: track 0.00 -> 89.1 mm
- net Net-(C12-Pad2): track 0.00 -> 55.6 mm
- net Net-(C10-Pad1): track 0.00 -> 54.0 mm
- net Net-(C8-Pad1): track 0.00 -> 52.5 mm
- net /pre amp/jfet_g: track 0.00 -> 49.4 mm
- net /pre amp/jfet_s: track 0.00 -> 39.0 mm
- net /pre amp/vgnd_disc: track 0.00 -> 36.8 mm
- net Net-(RV1-Pad2): track 0.00 -> 35.2 mm
- net /pre amp/PA_OUT: track 0.00 -> 34.6 mm
- net /pre amp/jfet_d: track 0.00 -> 28.0 mm
- net Net-(C12-Pad1): track 0.00 -> 21.8 mm
- net Net-(R38-Pad1): track 0.00 -> 20.7 mm
- net Net-(C1-Pad1): track 0.00 -> 18.6 mm
- net Net-(C7-Pad2): track 0.00 -> 14.5 mm
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