File: circuit/modulo.kicad_pcb (KiCad board)
At the start: 2 copper layers, 302 x 135 mm, 201 parts, among them J1 JACK_MONO, J10 HOLE, J11 HOLE, J12 HOLE, J13 HOLE, J14 HOLE, J15 HOLE, J17 HOLE, J18 HOLE, J19 HOLE, J2 Barrel_Jack_Switch, J24 HOLE, J25 HOLE, J26 HOLE, J27 HOLE, J3 HOLE, J4 HOLE, J5 HOLE, J6 HOLE, J7 HOLE, J8 HOLE, J9 HOLE, Q1 MMBFJ201, Q2 BC547, Q3 BC557, Q4 BC547, Q5 BC557, SW1 OFF/ON, SW2 ROT_SW, SW3 Idss/Vp, SW4 disc/TLE2426, SW5 disc/TLE2426, U1 TLE2426, U10 AVR-ISP6, U11 74164, U12 TPA3136D2, U13 74164, U14 modulo-bus, U15 modulo-bus, U16 modulo-bus, U17 TLE2426, U18 DBG_UART, U19 TPS560430, U2 NE5532, U3 FV-1, U4 NE5532, U5 24LC32A, U6 modulo-bus, U7 LM1117, U8 modulo-bus, U9 ATMEGA8, Y1 32768Hz, Y2 8MHz

Commit message: AVR software started; small hardware problems fixed
Parts:
- R1: value 1 -> 15K
- R2, R9: value 1 -> 1M
- R8: value 1 -> 1K5
Connections:
- J10 pad 1: Net-(J10-Pad1) -> (no net)
- J11 pad 1: Net-(J11-Pad1) -> (no net)
- J12 pad 1: Net-(J12-Pad1) -> (no net)
- J13 pad 1: Net-(J13-Pad1) -> (no net)
- J14 pad 1: Net-(J14-Pad1) -> (no net)
- J15 pad 1: Net-(J15-Pad1) -> (no net)
- J17 pad 1: Net-(J17-Pad1) -> (no net)
- J18 pad 1: Net-(J18-Pad1) -> (no net)
- J19 pad 1: Net-(J19-Pad1) -> (no net)
- J24 pad 1: Net-(J24-Pad1) -> (no net)
- J25 pad 1: Net-(J25-Pad1) -> (no net)
- J26 pad 1: Net-(J26-Pad1) -> (no net)
- J27 pad 1: Net-(J27-Pad1) -> (no net)
- J3 pad 1: Net-(J3-Pad1) -> (no net)
- J4 pad 1: Net-(J4-Pad1) -> (no net)
- J5 pad 1: Net-(J5-Pad1) -> (no net)
- J6 pad 1: Net-(J6-Pad1) -> (no net)
- J7 pad 1: Net-(J7-Pad1) -> (no net)
- J8 pad 1: Net-(J8-Pad1) -> (no net)
- J9 pad 1: Net-(J9-Pad1) -> (no net)
- R16 pad 2: +3V3 -> GND
- U12 pad 13: Net-(U12-Pad13) -> (no net)
- U12 pad 5: Net-(U12-Pad5) -> (no net)
- U12 pad 6: Net-(U12-Pad6) -> (no net)
- U13 pad 10: Net-(U13-Pad10) -> (no net)
- U13 pad 11: Net-(U13-Pad11) -> (no net)
- U13 pad 12: Net-(U13-Pad12) -> (no net)
- U13 pad 13: Net-(U13-Pad13) -> (no net)
- U14 pad 10: Net-(U14-Pad10) -> (no net)
- U14 pad 11: Net-(U14-Pad11) -> (no net)
- U14 pad 12: Net-(U14-Pad12) -> (no net)
- U14 pad 13: Net-(U14-Pad13) -> (no net)
- U14 pad 14: Net-(U14-Pad14) -> (no net)
- U14 pad 15: Net-(U14-Pad15) -> (no net)
- U14 pad 16: Net-(U14-Pad16) -> (no net)
- U14 pad 17: Net-(U14-Pad17) -> (no net)
- U14 pad 18: Net-(U14-Pad18) -> (no net)
- U14 pad 19: Net-(U14-Pad19) -> (no net)
- U14 pad 2: Net-(U14-Pad2) -> (no net)
- U14 pad 20: Net-(U14-Pad20) -> (no net)
- U14 pad 21: Net-(U14-Pad21) -> (no net)
- U14 pad 4: Net-(U14-Pad4) -> (no net)
- U14 pad 5: Net-(U14-Pad5) -> (no net)
- U14 pad 8: Net-(U14-Pad8) -> (no net)
- U14 pad 9: Net-(U14-Pad9) -> (no net)
- U15 pad 16: Net-(U15-Pad16) -> (no net)
- U15 pad 17: Net-(U15-Pad17) -> (no net)
- U15 pad 18: Net-(U15-Pad18) -> (no net)
- U15 pad 19: Net-(U15-Pad19) -> (no net)
- U15 pad 2: Net-(U15-Pad2) -> (no net)
- U15 pad 3: Net-(U15-Pad3) -> (no net)
- U15 pad 4: Net-(U15-Pad4) -> (no net)
- U16 pad 10: Net-(U16-Pad10) -> (no net)
- U16 pad 11: Net-(U16-Pad11) -> (no net)
- U16 pad 12: Net-(U16-Pad12) -> (no net)
- U16 pad 13: Net-(U16-Pad13) -> (no net)
- U16 pad 14: Net-(U16-Pad14) -> (no net)
- U16 pad 15: Net-(U16-Pad15) -> (no net)
- U16 pad 2: Net-(U16-Pad2) -> (no net)
- U16 pad 20: Net-(U16-Pad20) -> (no net)
- U16 pad 21: Net-(U16-Pad21) -> (no net)
- U16 pad 4: Net-(U16-Pad4) -> (no net)
- U16 pad 5: Net-(U16-Pad5) -> (no net)
- U6 pad 10: Net-(U6-Pad10) -> (no net)
- U6 pad 11: Net-(U6-Pad11) -> (no net)
- U6 pad 12: Net-(U6-Pad12) -> (no net)
- U6 pad 13: Net-(U6-Pad13) -> (no net)
- U6 pad 14: Net-(U6-Pad14) -> (no net)
- U6 pad 15: Net-(U6-Pad15) -> (no net)
- U6 pad 2: Net-(U6-Pad2) -> (no net)
- U6 pad 20: Net-(U6-Pad20) -> (no net)
- U6 pad 21: Net-(U6-Pad21) -> (no net)
- U6 pad 4: Net-(U6-Pad4) -> (no net)
- U6 pad 5: Net-(U6-Pad5) -> (no net)
- U6 pad 6: Net-(U6-Pad6) -> (no net)
- U6 pad 7: Net-(U6-Pad7) -> (no net)
- U6 pad 8: Net-(U6-Pad8) -> (no net)
- U6 pad 9: Net-(U6-Pad9) -> (no net)
- U8 pad 16: Net-(U8-Pad16) -> (no net)
- U8 pad 17: Net-(U8-Pad17) -> (no net)
- U8 pad 18: Net-(U8-Pad18) -> (no net)
- U8 pad 19: Net-(U8-Pad19) -> (no net)
- U8 pad 2: Net-(U8-Pad2) -> (no net)
- U8 pad 4: Net-(U8-Pad4) -> (no net)
- U8 pad 6: Net-(U8-Pad6) -> (no net)
- U8 pad 7: Net-(U8-Pad7) -> (no net)
- U8 pad 8: Net-(U8-Pad8) -> (no net)
- U8 pad 9: Net-(U8-Pad9) -> (no net)
- U9 pad 1: Net-(U9-Pad1) -> (no net)
- U9 pad 2: Net-(U9-Pad2) -> (no net)
- U9 pad 30: Net-(U9-Pad30) -> (no net)
- U9 pad 32: Net-(U9-Pad32) -> (no net)
Routing:
- net +3V3: track 339.7 -> 329.6 mm

Commit message: made FV-1 prototype; converted kicad 5 files to kicad 6
Other:
- net class Default removed
