File: circuit/modulo3-powamp.kicad_pcb (KiCad board)
At the start: 2 copper layers, 84 x 52 mm, 45 parts, among them J1 HOLE, J2 HOLE, J3 HOLE, J4 HOLE, SW3 HEAD/AD, U1 DIFFAUDIO, U2 TPA3220, U5 PWR_CONN, U6 AMPCTRL

Commit message: ready to panelize
Parts:
- moved R12 1.91 mm to (62.9, 82.5)
- moved R10 1.91 mm to (65.4, 82.5)
Routing:
- net +5V: track 168.2 -> 194.0 mm, vias 1 -> 0
Changed lines of the file:
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@@
   )
   (footprint "myAmp:R_10MM" (layer "F.Cu")
-    (at 62.992 80.645 90)
+    (at 62.865 82.55 90)
     (property "Sheetfile" "modulo3-powamp.kicad_sch")
     (property "Sheetname" "")
@@
   )
   (footprint "myAmp:R_10MM" (layer "F.Cu")
-    (at 65.405 80.645 90)
+    (at 65.405 82.55 90)
     (property "Sheetfile" "modulo3-powamp.kicad_sch")
     (property "Sheetname" "")
@@
   (segment (start 120.01 67.31) (end 119.335 66.635) (width 2.1844) (layer "F.Cu") (net 2))
   (segment (start 114.82 62.16) (end 119.295 66.635) (width 2.1844) (layer "F.Cu") (net 2))
-  (segment (start 54.61 60.452) (end 54.61 84.328) (width 0.8128) (layer "F.Cu") (net 3))
+  (segment (start 54.61 80.137) (end 54.61 84.328) (width 0.8128) (layer "F.Cu") (net 3))
+  (segment (start 61.976 76.2) (end 59.309 73.533) (width 0.4064) (layer "F.Cu") (net 3))
   (segment (start 72.136 83.82) (end 70.485 85.471) (width 0.8128) (layer "F.Cu") (net 3))
   (segment (start 75.52 82.4484) (end 75.266336 82.4484) (width 0.8128) (layer "F.Cu") (net 3))
+  (segment (start 57.15 74.041) (end 57.15 75.565) (width 0.4064) (layer "F.Cu") (net 3))
   (segment (start 82.505 69.215) (end 84.659998 69.215) (width 0.9652) (layer "F.Cu") (net 3))
   (segment (start 84.47 84.1375) (end 82.9241 84.1375) (width 0.3048) (layer "F.Cu") (net 3))
   (segment (start 70.485 85.471) (end 70.485 85.725) (width 0.8128) (layer "F.Cu") (net 3))
   (segment (start 81.235 57.195) (end 81.235 67.945) (width 0.8128) (layer "F.Cu") (net 3))
-  (segment (start 68.326 87.884) (end 70.485 85.725) (width 0.8128) (layer "F.Cu") (net 3))
+  (segment (start 59.817 78.232) (end 59.817 79.375) (width 0.4064) (layer "F.Cu") (net 3))
+  (segment (start 75.266336 82.4484) (end 73.894736 83.82) (width 0.8128) (layer "F.Cu") (net 3))
+  (segment (start 57.658 73.533) (end 57.15 74.041) (width 0.4064) (layer "F.Cu") (net 3))
+  (segment (start 54.61 60.452) (end 54.61 80.137) (width 0.8128) (layer "F.Cu") (net 3))
   (segment (start 68.834 51.562) (end 59.182 51.562) (width 0.8128) (layer "F.Cu") (net 3))
-  (segment (start 75.266336 82.4484) (end 73.894736 83.82) (width 0.8128) (layer "F.Cu") (net 3))
+  (segment (start 57.15 75.565) (end 59.817 78.232) (width 0.4064) (layer "F.Cu") (net 3))
+  (segment (start 73.615 77.47) (end 69.85 77.47) (width 0.4064) (layer "F.Cu") (net 3))
   (segment (start 85.471 52.959) (end 81.235 57.195) (width 0.8128) (layer "F.Cu") (net 3))
   (segment (start 84.659998 69.215) (end 84.66 69.215002) (width 0.9652) (layer "F.Cu") (net 3))
   (segment (start 68.834 59.436) (end 68.834 51.562) (width 0.6604) (layer "F.Cu") (net 3))
+  (segment (start 59.182 51.562) (end 57.7296 53.0144) (width 0.8128) (layer "F.Cu") (net 3))
   (segment (start 79.125 84.455) (end 78.613 84.455) (width 0.8128) (layer "F.Cu") (net 3))
   (segment (start 85.725 53.213) (end 107.95 53.213) (width 0.8128) (layer "F.Cu") (net 3))
   (segment (start 82.3366 84.725) (end 81.235 84.725) (width 0.3048) (layer "F.Cu") (net 3))
-  (segment (start 58.166 87.884) (end 68.326 87.884) (width 0.8128) (layer "F.Cu") (net 3))
+  (segment (start 69.85 77.47) (end 68.58 76.2) (width 0.4064) (layer "F.Cu") (net 3))
   (segment (start 85.471 52.959) (end 85.725 53.213) (width 0.8128) (layer "F.Cu") (net 3))
   (segment (start 67.945 60.325) (end 68.834 59.436) (width 0.6604) (layer "F.Cu") (net 3))
@@
   (segment (start 78.613 84.455) (end 76.6064 82.4484) (width 0.8128) (layer "F.Cu") (net 3))
   (segment (start 85.471 52.959) (end 84.074 51.562) (width 0.8128) (layer "F.Cu") (net 3))
-  (segment (start 59.182 51.562) (end 57.7296 53.0144) (width 0.8128) (layer "F.Cu") (net 3))
+  (segment (start 57.7296 53.0144) (end 57.7296 57.3324) (width 0.8128) (layer "F.Cu") (net 3))
   (segment (start 80.1334 84.725) (end 81.235 84.725) (width 0.6096) (layer "F.Cu") (net 3))
   (segment (start 81.235 67.945) (end 82.505 69.215) (width 0.9652) (layer "F.Cu") (net 3))
   (segment (start 84.074 51.562) (end 68.834 51.562) (width 0.8128) (layer "F.Cu") (net 3))
-  (segment (start 57.7296 57.3324) (end 54.61 60.452) (width 0.8128) (layer "F.Cu") (net 3))
+  (segment (start 68.58 76.2) (end 61.976 76.2) (width 0.4064) (layer "F.Cu") (net 3))
+  (segment (start 66.675 89.535) (end 70.485 85.725) (width 0.8128) (layer "F.Cu") (net 3))
   (segment (start 79.8634 84.455) (end 80.1334 84.725) (width 0.6096) (layer "F.Cu") (net 3))
   (segment (start 117.977 54.483) (end 118.46 54) (width 0.8128) (layer "F.Cu") (net 3))
   (segment (start 73.894736 83.82) (end 72.136 83.82) (width 0.8128) (layer "F.Cu") (net 3))
-  (segment (start 54.61 84.328) (end 58.166 87.884) (width 0.8128) (layer "F.Cu") (net 3))
+  (segment (start 59.309 73.533) (end 57.658 73.533) (width 0.4064) (layer "F.Cu") (net 3))
+  (segment (start 59.817 89.535) (end 66.675 89.535) (width 0.8128) (layer "F.Cu") (net 3))
+  (segment (start 59.817 79.375) (end 59.055 80.137) (width 0.4064) (layer "F.Cu") (net 3))
   (segment (start 109.22 54.483) (end 117.977 54.483) (width 0.8128) (layer "F.Cu") (net 3))
   (segment (start 79.125 84.455) (end 79.8634 84.455) (width 0.6096) (layer "F.Cu") (net 3))
-  (segment (start 57.7296 53.0144) (end 57.7296 57.3324) (width 0.8128) (layer "F.Cu") (net 3))
+  (segment (start 59.055 80.137) (end 54.61 80.137) (width 0.4064) (layer "F.Cu") (net 3))
+  (segment (start 54.61 84.328) (end 59.817 89.535) (width 0.8128) (layer "F.Cu") (net 3))
+  (segment (start 57.7296 57.3324) (end 54.61 60.452) (width 0.8128) (layer "F.Cu") (net 3))
   (segment (start 84.47 71.4375) (end 84.47 69.405002) (width 0.3048) (layer "F.Cu") (net 3))
   (segment (start 76.6064 82.4484) (end 75.52 82.4484) (width 0.8128) (layer "F.Cu") (net 3))
   (segment (start 84.47 69.405002) (end 84.66 69.215002) (width 0.3048) (layer "F.Cu") (net 3))
   (segment (start 82.9241 84.1375) (end 82.3366 84.725) (width 0.3048) (layer "F.Cu") (net 3))
-  (via (at 75.52 82.4484) (size 0.8) (drill 0.4) (layers "F.Cu" "B.Cu") (net 3))
-  (segment (start 73.615 77.47) (end 73.615 80.5434) (width 0.8128) (layer "B.Cu") (net 3))
-  (segment (start 73.615 80.5434) (end 75.52 82.4484) (width 0.8128) (layer "B.Cu") (net 3))
   (segment (start 91.97 71.4375) (end 93.176439 71.4375) (width 0.3048) (layer "F.Cu") (net 4))
   (segment (start 93.176439 71.4375) (end 94.488 70.125939) (width 0.3048) (layer "F.Cu") (net 4))
@@
   (segment (start 56.337699 61.264301) (end 56.337699 67.807699) (width 0.508) (layer "F.Cu") (net 12))
   (segment (start 56.337699 67.807699) (end 58.42 69.89) (width 0.508) (layer "F.Cu") (net 12))
-  (segment (start 59.015 74.89) (end 58.42 74.89) (width 0.3048) (layer "F.Cu") (net 13))
-  (segment (start 84.47 80.3275) (end 64.4525 80.3275) (width 0.3048) (layer "F.Cu") (net 13))
-  (segment (start 64.4525 80.3275) (end 59.015 74.89) (width 0.3048) (layer "F.Cu") (net 13))
-  (segment (start 59.19 57.269) (end 55.523901 60.935099) (width 0.508) (layer "F.Cu") (net 14))
-  (segment (start 59.19 54) (end 59.19 57.269) (width 0.508) (layer "F.Cu") (net 14))
+  (segment (start 84.47 80.3275) (end 63.1825 80.3275) (width 0.3048) (layer "F.Cu") (net 13))
+  (segment (start 58.42 75.565) (end 58.42 74.89) (width 0.3048) (layer "F.Cu") (net 13))
+  (segment (start 63.1825 80.3275) (end 58.42 75.565) (width 0.3048) (layer "F.Cu") (net 13))
+  (segment (start 58.674 57.785) (end 55.523901 60.935099) (width 0.508) (layer "F.Cu") (net 14))
   (segment (start 55.523901 75.883901) (end 58.42 78.78) (width 0.508) (layer "F.Cu") (net 14))
   (segment (start 55.523901 60.935099) (end 55.523901 75.883901) (width 0.508) (layer "F.Cu") (net 14))
+  (segment (start 58.674 54.516) (end 58.674 57.785) (width 0.508) (layer "F.Cu") (net 14))
+  (segment (start 59.19 54) (end 58.674 54.516) (width 0.508) (layer "F.Cu") (net 14))
   (segment (start 58.42 83.78) (end 61.2375 80.9625) (width 0.3048) (layer "F.Cu") (net 15))
   (segment (start 61.2375 80.9625) (end 84.47 80.9625) (width 0.3048) (layer "F.Cu") (net 15))
@@
   (segment (start 81.235 86.725) (end 80.3874 86.725) (width 0.6096) (layer "F.Cu") (net 30))
   (segment (start 84.47 84.7725) (end 83.4067 84.7725) (width 0.3048) (layer "F.Cu") (net 30))
+  (segment (start 62.865 77.47) (end 63.246 77.089) (width 0.6604) (layer "F.Cu") (net 31))
+  (segment (start 65.024 77.089) (end 65.405 77.47) (width 0.6604) (layer "F.Cu") (net 31))
+  (segment (start 67.31 77.47) (end 65.405 77.47) (width 0.3048) (layer "F.Cu") (net 31))
+  (segment (start 69.5325 79.6925) (end 67.31 77.47) (width 0.3048) (layer "F.Cu") (net 31))
+  (segment (start 63.246 77.089) (end 65.024 77.089) (width 0.6604) (layer "F.Cu") (net 31))
   (segment (start 84.47 79.6925) (end 69.5325 79.6925) (width 0.3048) (layer "F.Cu") (net 31))
-  (segment (start 62.992 75.565) (end 65.405 75.565) (width 0.6604) (layer "F.Cu") (net 31))
-  (segment (start 69.5325 79.6925) (end 65.405 75.565) (width 0.3048) (layer "F.Cu") (net 31))
   (segment (start 57.15 64.897) (end 60.452 61.595) (width 0.6096) (layer "F.Cu") (net 32))
   (segment (start 84.47 77.1525) (end 81.1657 77.1525) (width 0.3048) (layer "F.Cu") (net 32))
