File: circuit/modulo3-powamp.kicad_pcb (KiCad board)
At the start: 2 copper layers, 84 x 52 mm, 45 parts, among them J1 HOLE, J2 HOLE, J3 HOLE, J4 HOLE, SW3 HEAD/AD, U1 DIFFAUDIO, U2 TPA3220, U5 PWR_CONN, U6 AMPCTRL

Commit message: attempt to send to fab: part II
Other:
- board text added: "2023/04/16"
- board text removed: "2023/03/19"
Changed lines of the file:
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@@
     (effects (font (size 1.9 1.9) (thickness 0.3)))
   )
-  (gr_text "2023/03/19" (at 68 97) (layer "F.SilkS")
+  (gr_text "2023/04/16" (at 68 97) (layer "F.SilkS")
     (effects (font (size 2 2) (thickness 0.3)))
   )
